File: kicad/camera-gpio-interface-pcb.kicad_pcb (KiCad board)
At the start: 2 copper layers, 0 parts

Commit message: Initial v1.0 pcb layout
Parts:
- added C1001: 1uF, Capacitor_SMD:C_0402_1005Metric, F.Cu at (109.0, 82.5)
- added C1002: 1uF, Capacitor_SMD:C_0402_1005Metric, F.Cu at (111.0, 82.5)
- added C1101: 470pF, Capacitor_SMD:C_0402_1005Metric, F.Cu at (136.5, 114.2)
- added C1102: 470pF, Capacitor_SMD:C_0402_1005Metric, F.Cu at (139.5, 114.2)
- added C1103: 100nF, Capacitor_SMD:C_0402_1005Metric, F.Cu at (135.5, 112.0)
- added C1201: 100nF, Capacitor_SMD:C_0402_1005Metric, F.Cu at (161.0, 80.8)
- added C1202: 100nF, Capacitor_SMD:C_0402_1005Metric, F.Cu at (153.0, 80.8)
- added C1203: 100nF, Capacitor_SMD:C_0402_1005Metric, F.Cu at (148.2, 80.8)
- added C1401: 100nF, Capacitor_SMD:C_0402_1005Metric, F.Cu at (186.0, 80.8)
- added C1402: 100nF, Capacitor_SMD:C_0402_1005Metric, F.Cu at (178.0, 80.8)
- added C1403: 100nF, Capacitor_SMD:C_0402_1005Metric, F.Cu at (173.2, 80.8)
- added C401: 100nF, Capacitor_SMD:C_0402_1005Metric, F.Cu at (162.0, 108.0)
- added C501: 4.7uF, Capacitor_SMD:C_0402_1005Metric, F.Cu at (184.0, 85.0)
- added C502: 100nF, Capacitor_SMD:C_0402_1005Metric, F.Cu at (184.0, 105.5)
- added C503: 100nF, Capacitor_SMD:C_0402_1005Metric, F.Cu at (184.0, 99.0)
- added C504: 100nF, Capacitor_SMD:C_0402_1005Metric, F.Cu at (184.0, 92.5)
- added C505: 100nF, Capacitor_SMD:C_0402_1005Metric, F.Cu at (184.0, 86.0)
- added C701: 100nF, Capacitor_SMD:C_0402_1005Metric, F.Cu at (136.0, 80.8)
- added C702: 100nF, Capacitor_SMD:C_0402_1005Metric, F.Cu at (128.0, 80.8)
- added C703: 100nF, Capacitor_SMD:C_0402_1005Metric, F.Cu at (123.2, 80.8)
- added C901: 100nF, Capacitor_SMD:C_0402_1005Metric, F.Cu at (102.5, 93.2)
- added D1201: APHHS1005CGCK, orb_weaver_smd:LED_0402-1005_KNB, F.Cu at (153.0, 85.8)
- added D1401: APHHS1005CGCK, orb_weaver_smd:LED_0402-1005_KNB, F.Cu at (178.0, 85.8)
- added D201: APHHS1005CGCK, orb_weaver_smd:LED_0402-1005_KNB, F.Cu at (110.0, 84.1)
- added D301: APHHS1005CGCK, orb_weaver_smd:LED_0402-1005_KNB, F.Cu at (126.0, 110.0)
- added D302: APHHS1005CGCK, orb_weaver_smd:LED_0402-1005_KNB, F.Cu at (150.0, 110.0)
- added D401: APHHS1005CGCK, orb_weaver_smd:LED_0402-1005_KNB, F.Cu at (174.0, 110.0)
- added D701: APHHS1005CGCK, orb_weaver_smd:LED_0402-1005_KNB, F.Cu at (128.0, 85.8)
- added D901: MBR120VLSFT1G, orb_weaver_smd:SOD-123FL, F.Cu at (111.0, 90.0)
- added FID101: Fiducial 1mm Mask 2mm, Fiducial:Fiducial_1mm_Mask2mm, F.Cu at (105.0, 77.0)
- added FID102: Fiducial 1mm Mask 2mm, Fiducial:Fiducial_1mm_Mask2mm, F.Cu at (195.0, 77.0)
- added FID103: Fiducial 1mm Mask 2mm, Fiducial:Fiducial_1mm_Mask2mm, F.Cu at (105.0, 113.0)
- added H101: Mounting Hole 3.2mm M3, MountingHole:MountingHole_3.2mm_M3, F.Cu at (105.0, 70.0)
- added H102: Mounting Hole 3.2mm M3, MountingHole:MountingHole_3.2mm_M3, F.Cu at (195.0, 70.0)
- added H103: Mounting Hole 3.2mm M3, MountingHole:MountingHole_3.2mm_M3, F.Cu at (195.0, 120.0)
- added H104: Mounting Hole 3.2mm M3, MountingHole:MountingHole_3.2mm_M3, F.Cu at (105.0, 120.0)
- added J1201: TBH-1x06-3.5mm, orb_weaver_tht:PhoenixContact_MCV_1,5_6-G-3.5_1x06_P3.50mm_Vertical, F.Cu at (150.0, 71.0)
- added J1401: TBH-1x06-3.5mm, orb_weaver_tht:PhoenixContact_MCV_1,5_6-G-3.5_1x06_P3.50mm_Vertical, F.Cu at (175.0, 71.0)
- added J301: HL-BNC-KHDA, orb_weaver_connectors:CONN_BNC_HL-BNC-KHDA, F.Cu at (126.0, 118.0)
- added J302: HL-BNC-KHDA, orb_weaver_connectors:CONN_BNC_HL-BNC-KHDA, F.Cu at (150.0, 118.0)
- added J401: HL-BNC-KHDA, orb_weaver_connectors:CONN_BNC_HL-BNC-KHDA, F.Cu at (174.0, 118.0)
- added J402: HL-BNC-KHDA, orb_weaver_connectors:CONN_BNC_HL-BNC-KHDA, F.Cu at (126.0, 94.0)
- added J403: HL-BNC-KHDA, orb_weaver_connectors:CONN_BNC_HL-BNC-KHDA, F.Cu at (150.0, 94.0)
- added J404: HL-BNC-KHDA, orb_weaver_connectors:CONN_BNC_HL-BNC-KHDA, F.Cu at (174.0, 94.0)
- added J501: FH12-50S-0.5SVA(54), orb_weaver_connectors:Hirose_FH12-50S-0.5SVA_1x50-4MP_P0.5mm_Vertical, F.Cu at (194.0, 99.0)
- added J701: TBH-1x06-3.5mm, orb_weaver_tht:PhoenixContact_MCV_1,5_6-G-3.5_1x06_P3.50mm_Vertical, F.Cu at (125.0, 71.0)
- added J901: USB-C, orb_weaver_connectors:USB_C_Receptacle_GCT_USB4145-03-0070-C_16P_Vertical, F.Cu at (106.0, 94.0)
- added R1101: 100k, Resistor_SMD:R_0402_1005Metric, F.Cu at (137.5, 114.2)
- added R1102: 100k, Resistor_SMD:R_0402_1005Metric, F.Cu at (138.5, 114.2)
- added R1103: 4.7k, Resistor_SMD:R_0402_1005Metric, F.Cu at (135.5, 114.2)
- added R1104: 4.7k, Resistor_SMD:R_0402_1005Metric, F.Cu at (140.5, 114.2)
- added R1105: 100k, Resistor_SMD:R_0402_1005Metric, F.Cu at (136.5, 110.0)
- added R1106: 100k, Resistor_SMD:R_0402_1005Metric, F.Cu at (139.5, 110.0)
- added R1107: 100, Resistor_SMD:R_0402_1005Metric, F.Cu at (136.5, 108.0)
- added R1108: 100, Resistor_SMD:R_0402_1005Metric, F.Cu at (139.5, 108.0)
- added R1201: 1k, Resistor_SMD:R_0402_1005Metric, F.Cu at (151.8, 77.0)
- added R1202: 4.7k, Resistor_SMD:R_0402_1005Metric, F.Cu at (147.2, 80.8)
- added R1203: 820, Resistor_SMD:R_0402_1005Metric, F.Cu at (155.2, 77.0)
- added R1204: 220, Resistor_SMD:R_0603_1608Metric, F.Cu at (159.2, 77.5)
- added R1205: 470, Resistor_SMD:R_0603_1608Metric, F.Cu at (151.8, 84.2)
- added R1206: 680, Resistor_SMD:R_0402_1005Metric, F.Cu at (153.0, 83.8)
- added R1207: 100, Resistor_SMD:R_0402_1005Metric, F.Cu at (156.5, 80.8)
- added R1208: 100, Resistor_SMD:R_0402_1005Metric, F.Cu at (149.5, 83.8)
- added R1209: 100, Resistor_SMD:R_0402_1005Metric, F.Cu at (151.8, 80.8)
- added R1210: 100, Resistor_SMD:R_0402_1005Metric, F.Cu at (157.5, 80.8)
- added R1211: 100, Resistor_SMD:R_0402_1005Metric, F.Cu at (150.5, 83.8)
- added R1401: 1k, Resistor_SMD:R_0402_1005Metric, F.Cu at (176.8, 77.0)
- added R1402: 4.7k, Resistor_SMD:R_0402_1005Metric, F.Cu at (172.2, 80.8)
- added R1403: 820, Resistor_SMD:R_0402_1005Metric, F.Cu at (180.2, 77.0)
- added R1404: 220, Resistor_SMD:R_0603_1608Metric, F.Cu at (184.2, 77.5)
- added R1405: 470, Resistor_SMD:R_0603_1608Metric, F.Cu at (176.8, 84.2)
- added R1406: 680, Resistor_SMD:R_0402_1005Metric, F.Cu at (178.0, 83.8)
- added R1407: 100, Resistor_SMD:R_0402_1005Metric, F.Cu at (181.5, 80.8)
- added R1408: 100, Resistor_SMD:R_0402_1005Metric, F.Cu at (174.5, 83.8)
- added R1409: 100, Resistor_SMD:R_0402_1005Metric, F.Cu at (176.8, 80.8)
- added R1410: 100, Resistor_SMD:R_0402_1005Metric, F.Cu at (182.5, 80.8)
- added R1411: 100, Resistor_SMD:R_0402_1005Metric, F.Cu at (175.5, 83.8)
- added R201: 680, Resistor_SMD:R_0402_1005Metric, F.Cu at (112.0, 84.0)
- added R301: 680, Resistor_SMD:R_0402_1005Metric, F.Cu at (126.0, 108.0)
- added R302: 680, Resistor_SMD:R_0402_1005Metric, F.Cu at (150.0, 108.0)
- added R401: 680, Resistor_SMD:R_0402_1005Metric, F.Cu at (174.0, 108.0)
- added R402: 470, Resistor_SMD:R_0603_1608Metric, F.Cu at (165.0, 107.0)
- added R403: 100, Resistor_SMD:R_0402_1005Metric, F.Cu at (165.0, 105.0)
- added R501: 10k, Resistor_SMD:R_0402_1005Metric, F.Cu at (186.0, 105.5)
- added R502: 10k, Resistor_SMD:R_0402_1005Metric, F.Cu at (186.0, 99.0)
- added R503: 10k, Resistor_SMD:R_0402_1005Metric, F.Cu at (186.0, 92.5)
- added R504: 10k, Resistor_SMD:R_0402_1005Metric, F.Cu at (186.0, 86.0)
- added R505: 100, Resistor_SMD:R_0402_1005Metric, F.Cu at (188.2, 110.8)
- added R506: 100, Resistor_SMD:R_0402_1005Metric, F.Cu at (190.2, 110.2)
- added R507: 100, Resistor_SMD:R_0402_1005Metric, F.Cu at (190.2, 109.2)
- added R508: 100, Resistor_SMD:R_0402_1005Metric, F.Cu at (188.2, 108.8)
- added R509: 100, Resistor_SMD:R_0402_1005Metric, F.Cu at (188.2, 107.8)
- added R510: 100, Resistor_SMD:R_0402_1005Metric, F.Cu at (190.2, 107.2)
- added R511: 100, Resistor_SMD:R_0402_1005Metric, F.Cu at (190.2, 106.2)
- added R512: 100, Resistor_SMD:R_0402_1005Metric, F.Cu at (188.2, 105.8)
- added R513: 100, Resistor_SMD:R_0402_1005Metric, F.Cu at (188.2, 104.8)
- added R514: 100, Resistor_SMD:R_0402_1005Metric, F.Cu at (190.2, 104.2)
- added R515: 100, Resistor_SMD:R_0402_1005Metric, F.Cu at (190.2, 103.2)
- added R516: 100, Resistor_SMD:R_0402_1005Metric, F.Cu at (188.2, 102.8)
- added R517: 100, Resistor_SMD:R_0402_1005Metric, F.Cu at (188.2, 101.8)
- added R518: 100, Resistor_SMD:R_0402_1005Metric, F.Cu at (190.2, 101.2)
- added R519: 100, Resistor_SMD:R_0402_1005Metric, F.Cu at (190.2, 100.2)
- added R520: 100, Resistor_SMD:R_0402_1005Metric, F.Cu at (188.2, 99.8)
- added R521: 100, Resistor_SMD:R_0402_1005Metric, F.Cu at (190.2, 98.2)
- added R522: 100, Resistor_SMD:R_0402_1005Metric, F.Cu at (188.2, 97.8)
- added R523: 100, Resistor_SMD:R_0402_1005Metric, F.Cu at (188.2, 96.8)
- added R524: 100, Resistor_SMD:R_0402_1005Metric, F.Cu at (190.2, 96.2)
- added R525: 100, Resistor_SMD:R_0402_1005Metric, F.Cu at (190.2, 95.2)
- added R526: 100, Resistor_SMD:R_0402_1005Metric, F.Cu at (188.2, 94.8)
- added R527: 100, Resistor_SMD:R_0402_1005Metric, F.Cu at (188.2, 93.8)
- added R528: 100, Resistor_SMD:R_0402_1005Metric, F.Cu at (190.2, 93.2)
- added R529: 100, Resistor_SMD:R_0402_1005Metric, F.Cu at (190.2, 92.2)
- added R530: 100, Resistor_SMD:R_0402_1005Metric, F.Cu at (188.2, 91.8)
- added R531: 100, Resistor_SMD:R_0402_1005Metric, F.Cu at (188.2, 90.8)
- added R532: 100, Resistor_SMD:R_0402_1005Metric, F.Cu at (190.2, 90.2)
- added R533: 100, Resistor_SMD:R_0402_1005Metric, F.Cu at (190.2, 89.2)
- added R534: 100, Resistor_SMD:R_0402_1005Metric, F.Cu at (188.2, 88.8)
- added R535: 100, Resistor_SMD:R_0402_1005Metric, F.Cu at (188.2, 87.8)
- added R536: 100, Resistor_SMD:R_0402_1005Metric, F.Cu at (190.2, 87.2)
- added R701: 1k, Resistor_SMD:R_0402_1005Metric, F.Cu at (126.8, 77.0)
- added R702: 4.7k, Resistor_SMD:R_0402_1005Metric, F.Cu at (122.2, 80.8)
- added R703: 820, Resistor_SMD:R_0402_1005Metric, F.Cu at (130.2, 77.0)
- added R704: 220, Resistor_SMD:R_0603_1608Metric, F.Cu at (134.2, 77.5)
- added R705: 470, Resistor_SMD:R_0603_1608Metric, F.Cu at (126.8, 84.2)
- added R706: 680, Resistor_SMD:R_0402_1005Metric, F.Cu at (128.0, 83.8)
- added R707: 100, Resistor_SMD:R_0402_1005Metric, F.Cu at (131.5, 80.8)
- added R708: 100, Resistor_SMD:R_0402_1005Metric, F.Cu at (124.5, 83.8)
- added R709: 100, Resistor_SMD:R_0402_1005Metric, F.Cu at (126.8, 80.8)
- added R710: 100, Resistor_SMD:R_0402_1005Metric, F.Cu at (132.5, 80.8)
- added R711: 100, Resistor_SMD:R_0402_1005Metric, F.Cu at (125.5, 83.8)
- added R901: 5.1k, Resistor_SMD:R_0402_1005Metric, F.Cu at (102.5, 94.8)
- added R902: 5.1k, Resistor_SMD:R_0402_1005Metric, F.Cu at (109.5, 92.2)
- added U1001: TPS73733QDRBRQ1, orb_weaver_smd:TPS737Q1, F.Cu at (110.0, 80.0)
- added U1101: SN74LVC2G17DRYR, orb_weaver_smd:DRY6, F.Cu at (138.0, 112.0)
- added U1201: SN74LVC2G17DRYR, orb_weaver_smd:DRY6, F.Cu at (150.0, 80.8)
- added U1202: SN74LVC1G125DRYR, orb_weaver_smd:DRY6, F.Cu at (159.2, 80.8)
- added U1203: SN74LVC1G07DRYR, orb_weaver_smd:DRY6, F.Cu at (154.8, 80.8)
- added U1204: USBLC6-2P6, orb_weaver_smd:USBLC6-2P6_SOT-666, F.Cu at (157.0, 77.5)
- added U1205: USBLC6-2P6, orb_weaver_smd:USBLC6-2P6_SOT-666, F.Cu at (150.0, 77.5)
- added U1401: SN74LVC2G17DRYR, orb_weaver_smd:DRY6, F.Cu at (175.0, 80.8)
- added U1402: SN74LVC1G125DRYR, orb_weaver_smd:DRY6, F.Cu at (184.2, 80.8)
- added U1403: SN74LVC1G07DRYR, orb_weaver_smd:DRY6, F.Cu at (179.8, 80.8)
- added U1404: USBLC6-2P6, orb_weaver_smd:USBLC6-2P6_SOT-666, F.Cu at (182.0, 77.5)
- added U1405: USBLC6-2P6, orb_weaver_smd:USBLC6-2P6_SOT-666, F.Cu at (175.0, 77.5)
- added U301: USBLC6-2P6, orb_weaver_smd:USBLC6-2P6_SOT-666, F.Cu at (138.0, 119.0)
- added U401: SN74LVC1G125DRYR, orb_weaver_smd:DRY6, F.Cu at (162.0, 106.0)
- added U402: USBLC6-2P6, orb_weaver_smd:USBLC6-2P6_SOT-666, F.Cu at (138.0, 95.0)
- added U403: USBLC6-2P6, orb_weaver_smd:USBLC6-2P6_SOT-666, F.Cu at (177.0, 106.0)
- added U501: SN74LV541ARKSR, orb_weaver_smd:Texas_RKS0020A_VQFN-20-1EP_2.5x4.5mm_P0.5mm_EP1x3mm, F.Cu at (185.0, 108.8)
- added U502: SN74LV541ARKSR, orb_weaver_smd:Texas_RKS0020A_VQFN-20-1EP_2.5x4.5mm_P0.5mm_EP1x3mm, F.Cu at (185.0, 102.2)
- added U503: SN74LV541ARKSR, orb_weaver_smd:Texas_RKS0020A_VQFN-20-1EP_2.5x4.5mm_P0.5mm_EP1x3mm, F.Cu at (185.0, 95.8)
- added U504: SN74LV541ARKSR, orb_weaver_smd:Texas_RKS0020A_VQFN-20-1EP_2.5x4.5mm_P0.5mm_EP1x3mm, F.Cu at (185.0, 89.2)
- added U701: SN74LVC2G17DRYR, orb_weaver_smd:DRY6, F.Cu at (125.0, 80.8)
- added U702: SN74LVC1G125DRYR, orb_weaver_smd:DRY6, F.Cu at (134.2, 80.8)
- added U703: SN74LVC1G07DRYR, orb_weaver_smd:DRY6, F.Cu at (129.8, 80.8)
- added U704: USBLC6-2P6, orb_weaver_smd:USBLC6-2P6_SOT-666, F.Cu at (132.0, 77.5)
- added U705: USBLC6-2P6, orb_weaver_smd:USBLC6-2P6_SOT-666, F.Cu at (125.0, 77.5)
- added U901: USBLC6-2P6, orb_weaver_smd:USBLC6-2P6_SOT-666, F.Cu at (111.0, 94.0)
Routing:
- net /GND: track 0.00 -> 314.5 mm, vias 0 -> 48
- net /+3.3V: track 0.00 -> 131.6 mm, vias 0 -> 28
- net /+5V: track 0.00 -> 35.1 mm, vias 0 -> 9
- net /power/usb2_vertical/VBUS: track 0.00 -> 18.7 mm, vias 0 -> 3
- net /blackfly_s_gpio_channel_mcv6_vertical2/L1: track 0.00 -> 11.7 mm
- net /blackfly_s_gpio_channel_mcv6_vertical1/L1: track 0.00 -> 11.7 mm
- net /blackfly_s_gpio_channel_mcv6_vertical/L1: track 0.00 -> 11.7 mm
- net /blackfly_s_gpio_channel_mcv6_vertical/L2: track 0.00 -> 10.9 mm
- net /blackfly_s_gpio_channel_mcv6_vertical1/L2: track 0.00 -> 10.9 mm
- net /blackfly_s_gpio_channel_mcv6_vertical2/L2: track 0.00 -> 10.9 mm
- net /blackfly_s_gpio_channel_mcv6_vertical2/L0: track 0.00 -> 10.7 mm
- net /blackfly_s_gpio_channel_mcv6_vertical1/L0: track 0.00 -> 10.7 mm
- net /blackfly_s_gpio_channel_mcv6_vertical/L0: track 0.00 -> 10.7 mm
- net /blackfly_s_gpio_channel_mcv6_vertical2/L3: track 0.00 -> 9.78 mm
- net /blackfly_s_gpio_channel_mcv6_vertical1/L3: track 0.00 -> 9.78 mm
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Other:
- board outline added: 100 x 60 mm
- copper layers 2 -> 4
- board text added: "+3.3V"
- board text added: "+5V"
- board text added: "50-PIN"
- board text added: "BLK"
- board text added: "BLU"
- board text added: "BRN"
- board text added: "CAMERA 1"
- board text added: "CAMERA 1 OUT"
- board text added: "CAMERA 2"
- board text added: "CAMERA 2 OUT"
- board text added: "CAMERA 3"
- board text added: "CAMERA 3 OUT"
- board text added: "GRN"
- board text added: "RED"
- board text added: "SYNC IN"
- board text added: "SYNC OUT"
- board text added: "TRIG IN"
- board text added: "WHT"
- board text added: "camera-gpio-interface-pcb v1.0 09/26"
