File: kicad/camera-gpio-interface-pcb.kicad_pcb (KiCad board)
At the start: 4 copper layers, 100 x 60 mm, 158 parts, among them J1201 TBH-1x06-3.5mm, J1401 TBH-1x06-3.5mm, J301 HL-BNC-KHDA, J302 HL-BNC-KHDA, J401 HL-BNC-KHDA, J402 HL-BNC-KHDA, J403 HL-BNC-KHDA, J404 HL-BNC-KHDA, J501 FH12-50S-0.5SVA(54), J701 TBH-1x06-3.5mm, J901 USB-C, U1001 TPS73733QDRBRQ1, U1101 SN74LVC2G17DRYR, U1201 SN74LVC2G17DRYR, U1202 SN74LVC1G125DRYR, U1203 SN74LVC1G07DRYR, U1204 USBLC6-2P6, U1205 USBLC6-2P6, U1401 SN74LVC2G17DRYR, U1402 SN74LVC1G125DRYR, U1403 SN74LVC1G07DRYR, U1404 USBLC6-2P6, U1405 USBLC6-2P6, U301 USBLC6-2P6, U401 SN74LVC1G125DRYR, U402 USBLC6-2P6, U403 USBLC6-2P6, U501 SN74LV541ARKSR, U502 SN74LV541ARKSR, U503 SN74LV541ARKSR, U504 SN74LV541ARKSR, U701 SN74LVC2G17DRYR, U702 SN74LVC1G125DRYR, U703 SN74LVC1G07DRYR, U704 USBLC6-2P6, U705 USBLC6-2P6, U901 USBLC6-2P6

Commit message: Found a routing solution
Parts:
- turned U402 to 90 degrees
Routing:
- net /+5V: track 35.1 -> 195.1 mm, vias 9 -> 14
- net /+3.3V: track 131.6 -> 238.4 mm, vias 28 -> 31
- net /SYNC_IN: track 8.23 -> 113.3 mm, vias 4 -> 9
- net /TRIG_IN: track 8.20 -> 99.4 mm, vias 4 -> 7
- net /CAM1_L1_INST: track 0.99 -> 71.6 mm, vias 1 -> 4
- net /CAM1_L2_INST: track 0.99 -> 69.7 mm, vias 1 -> 2
- net /CAM1_OUT_INST: track 0.99 -> 68.7 mm, vias 1 -> 2
- net /CAM1_L0_INST: track 0.99 -> 67.7 mm, vias 1 -> 4
- net /CAM1_L3_INST: track 0.99 -> 63.2 mm, vias 1 -> 3
- net /TRIG_IN_INST: track 1.00 -> 48.6 mm, vias 1 -> 2
- net /SYNC_IN_INST: track 1.00 -> 47.8 mm, vias 1 -> 2
- net /CAM2_L1_INST: track 0.99 -> 44.0 mm, vias 1 -> 2
- net /CAM2_OUT_INST: track 0.99 -> 43.8 mm, vias 1 -> 2
- net /CAM2_L2_INST: track 0.99 -> 41.7 mm, vias 1 -> 2
- net /CAM2_L0_INST: track 0.99 -> 38.2 mm, vias 1 -> 3
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- added copper zone on B.Cu, net /GND
- added copper zone on In1.Cu, net /GND

Commit message: Update with changes after fixing kicad-lib scripts
Routing:
- net /SYNC_IN: track 113.3 -> 112.3 mm, vias 9 -> 8
- net /power/usb2_vertical/USB_D+: vias 2 -> 0
- net /CAM2_L3_INST: vias 3 -> 2
- net /CAM2_L0_INST: vias 3 -> 2
- net /CAM1_L3_INST: vias 3 -> 2
Changed lines of the file:
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@@
 		(net "/power/usb2_vertical/USB_D+")
 	)
-	(via
-		(at 106.5 93.5)
-		(size 0.6)
-		(drill 0.3)
-		(layers "F.Cu" "B.Cu")
-		(net "/power/usb2_vertical/USB_D+")
-	)
-	(via
-		(at 105.5 94.5)
-		(size 0.6)
-		(drill 0.3)
-		(layers "F.Cu" "B.Cu")
-		(net "/power/usb2_vertical/USB_D+")
-	)
 	(segment
 		(start 107.5 92)
@@
 	)
 	(segment
-		(start 139.5 109)
-		(end 138.5 109)
-		(width 0.2)
-		(layer "F.Cu")
-		(net "/SYNC_IN")
-	)
-	(segment
 		(start 147.992 108.51)
 		(end 148.527 107.975)
@@
 	)
 	(via
-		(at 138.5 109)
-		(size 0.6)
-		(drill 0.3)
-		(layers "F.Cu" "B.Cu")
-		(net "/SYNC_IN")
-	)
-	(via
 		(at 137.88 81.0905)
 		(size 0.6)
@@
 		(net "/CAM2_L3_INST")
 	)
-	(via
-		(at 157.5 82.25)
-		(size 0.6)
-		(drill 0.3)
-		(layers "F.Cu" "B.Cu")
-		(net "/CAM2_L3_INST")
-	)
 	(segment
 		(start 170.047 93.6763)
@@
 	)
 	(via
-		(at 156.5 82.25)
-		(size 0.6)
-		(drill 0.3)
-		(layers "F.Cu" "B.Cu")
-		(net "/CAM2_L0_INST")
-	)
-	(via
 		(at 179.859 103.684)
 		(size 0.6)
@@
 		(size 0.6)
 		(drill 0.3)
-		(layers "F.Cu" "B.Cu")
-		(net "/CAM1_L3_INST")
-	)
-	(via
-		(at 132.5 82.25)
-		(size 0.6)
-		(drill 0.3)

Commit message: Finished v1.0 changes
Routing:
- net /GND: vias 58 -> 59
- added copper zone on F.Cu, net /GND
- added copper zone on In2.Cu, net /GND
Other:
- board text added: "CAM1 OUT"
- board text added: "CAM2 OUT"
- board text added: "CAM3 OUT"
- board text added: "USB 5V"
- board text removed: "CAMERA 1 OUT"
- board text removed: "CAMERA 2 OUT"
- board text removed: "CAMERA 3 OUT"

Commit message: Regenerate schematics
Connections:
- net Net-(D1201-A) renamed /blackfly_s_gpio_channel_mcv6_vertical1/LED_A
- net Net-(D1401-A) renamed /blackfly_s_gpio_channel_mcv6_vertical2/LED_A
- net Net-(D701-A) renamed /blackfly_s_gpio_channel_mcv6_vertical/LED_A
Routing:
- net Net-(D701-A): track 0.00 -> 1.04 mm
- net Net-(D1401-A): track 0.00 -> 1.04 mm
- net Net-(D1201-A): track 0.00 -> 1.04 mm
- net /blackfly_s_gpio_channel_mcv6_vertical2/LED_A: track 1.04 -> 0.00 mm
- net /blackfly_s_gpio_channel_mcv6_vertical1/LED_A: track 1.04 -> 0.00 mm
- net /blackfly_s_gpio_channel_mcv6_vertical/LED_A: track 1.04 -> 0.00 mm
Changed lines of the file:
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@@
 			(layers "F.Cu" "F.Mask" "F.Paste")
 			(roundrect_rratio 0.25)
-			(net "Net-(D1201-A)")
+			(net "/blackfly_s_gpio_channel_mcv6_vertical1/LED_A")
 			(pintype "passive")
 		)
@@
 			(size 0.7 0.5)
 			(layers "F.Cu" "F.Mask" "F.Paste")
-			(net "Net-(D701-A)")
+			(net "/blackfly_s_gpio_channel_mcv6_vertical/LED_A")
 			(pinfunction "A_2")
 			(pintype "passive")
@@
 			(layers "F.Cu" "F.Mask" "F.Paste")
 			(roundrect_rratio 0.25)
-			(net "Net-(D1401-A)")
+			(net "/blackfly_s_gpio_channel_mcv6_vertical2/LED_A")
 			(pintype "passive")
 		)
@@
 			(size 0.7 0.5)
 			(layers "F.Cu" "F.Mask" "F.Paste")
-			(net "Net-(D1401-A)")
+			(net "/blackfly_s_gpio_channel_mcv6_vertical2/LED_A")
 			(pinfunction "A_2")
 			(pintype "passive")
@@
 			(layers "F.Cu" "F.Mask" "F.Paste")
 			(roundrect_rratio 0.25)
-			(net "Net-(D701-A)")
+			(net "/blackfly_s_gpio_channel_mcv6_vertical/LED_A")
 			(pintype "passive")
 		)
@@
 			(size 0.7 0.5)
 			(layers "F.Cu" "F.Mask" "F.Paste")
-			(net "Net-(D1201-A)")
+			(net "/blackfly_s_gpio_channel_mcv6_vertical1/LED_A")
 			(pinfunction "A_2")
 			(pintype "passive")
@@
 	)
 	(group "blackfly_s_gpio_channel_mcv6_vertical_1"
-		(lib_id "orb_weaver_private:blackfly_s_gpio_channel_mcv6_vertical")
+		(lib_id "orb_weaver_blackfly_s_gpio_channel:blackfly_s_gpio_channel_mcv6_vertical")
 		(members "01249ea6-ec37-490c-85ab-aadbf7d54ab9" "050a3cbd-effb-4d6f-aec8-d16f08d1e55e"
 			"37383403-7e48-4736-b744-a3515263683a" "424a7bf7-8e51-463e-be8a-738b0f412350"
@@
 	)
 	(group "blackfly_s_gpio_channel_mcv6_vertical_3"
-		(lib_id "orb_weaver_private:blackfly_s_gpio_channel_mcv6_vertical")
+		(lib_id "orb_weaver_blackfly_s_gpio_channel:blackfly_s_gpio_channel_mcv6_vertical")
 		(members "09ed3c75-0a24-4094-b7ea-1973f4e8fefe" "0af2b6a6-87d3-4824-af12-de84e3514f38"
 			"1db0a239-dff6-48d5-97db-9cd88c83e1d6" "23c1d4ff-e2b3-48c4-83ba-025b3b7963e9"
@@
 	)
 	(group "blackfly_s_gpio_channel_mcv6_vertical_2"
-		(lib_id "orb_weaver_private:blackfly_s_gpio_channel_mcv6_vertical")
+		(lib_id "orb_weaver_blackfly_s_gpio_channel:blackfly_s_gpio_channel_mcv6_vertical")
 		(members "0bf0736f-8a6c-4cd9-9602-dde66dddd49c" "0c0f5b25-6f1b-465f-8bed-ee975f083adb"
 			"0ef06be0-1b31-491d-9eec-cf805311fd38" "12ee70a8-8364-44ec-b83f-4c13eeaaf00b"
