File: kicad/inputs.kicad_sch (KiCad schematic)
At the start: 0 parts

Commit message: Initial v1.0 pcb layout
Parts:
- added D301, D302: APHHS1005CGCK, orb_weaver_smd:LED_0402-1005_KNB, symbol orb_weaver_internal:All/OW-MISC-APHHS1005CGCK
- added J301, J302: HL-BNC-KHDA, orb_weaver_connectors:CONN_BNC_HL-BNC-KHDA, symbol orb_weaver_internal:All/OW-CONN-HL-BNC-KHDA
- added R301, R302: 680, Resistor_SMD:R_0402_1005Metric, symbol orb_weaver_internal:All/OW-PASS-RC0402FR-07680RL
- added U301: USBLC6-2P6, orb_weaver_smd:USBLC6-2P6_SOT-666, symbol orb_weaver_internal:All/OW-MISC-USBLC6-2P6
Connections:
- new net: D301.2 (A), R301.2
- new net: D302.2 (A), R302.2
- new net +5V: U301.5 (VBUS)
- new net GND: D301.1 (K), D302.1 (K), J301.2 (Shield), J302.2 (Shield), U301.2 (GND)
- new net SYNC_IN: R302.1
- new net SYNC_RAW: J302.1 (Signal), U301.3 (I/O2), U301.4 (I/O2)
- new net TRIG_IN: R301.1
- new net TRIG_RAW: J301.1 (Signal), U301.1 (I/O1), U301.6 (I/O1)
Other:
- added sheet logic_input_2ch_5v_schmitt_sn74lvc2g17 (logic_input_2ch_5v_schmitt_sn74lvc2g17.kicad_sch)
