File: kicad/camera-gpio-interface-pcb.kicad_sch (KiCad schematic)
At the start: 0 parts

Commit message: Add root level schematic sheets
Other:
- added sheet camera_1 (camera_1.kicad_sch)
- added sheet camera_2 (camera_2.kicad_sch)
- added sheet camera_3 (camera_3.kicad_sch)
- added sheet inputs (inputs.kicad_sch)
- added sheet instrument_port (instrument_port.kicad_sch)
- added sheet power (power.kicad_sch)
- added sheet sync_out (sync_out.kicad_sch)
- company: (none) -> Janelia Research Campus
- title: (none) -> camera-gpio-interface-pcb

Commit message: Initial v1.0 pcb layout
Parts:
- added FID101, FID102, FID103: Fiducial 1mm Mask 2mm, Fiducial:Fiducial_1mm_Mask2mm, symbol orb_weaver_internal:All/OW-MECH-FID-1MM-MASK2MM
- added H101, H102, H103, H104: Mounting Hole 3.2mm M3, MountingHole:MountingHole_3.2mm_M3, symbol orb_weaver_internal:All/OW-MECH-MH-3-2MM-M3
Other:
- sheet sync_out renamed outputs
- removed sheet camera_1
- removed sheet camera_2
- removed sheet camera_3
- removed sheet instrument_port
- added sheet blackfly_s_gpio_channel_mcv6_vertical (blackfly_s_gpio_channel_mcv6_vertical.kicad_sch)
- added sheet blackfly_s_gpio_channel_mcv6_vertical1 (blackfly_s_gpio_channel_mcv6_vertical.kicad_sch)
- added sheet blackfly_s_gpio_channel_mcv6_vertical2 (blackfly_s_gpio_channel_mcv6_vertical.kicad_sch)
- added sheet instrument_port_digital_50_dut_ffc_boundary_vertical (instrument_port_digital_50_dut_ffc_boundary_vertical.kicad_sch)
- sheet inputs ports: added +3.3V, +5V, GND, SYNC_IN, SYNC_IN_INST, TRIG_IN, TRIG_IN_INST; removed none
- sheet outputs: file sync_out.kicad_sch -> outputs.kicad_sch
- sheet outputs ports: added +3.3V, +5V, CAM1_OUT_BNC, CAM2_OUT_BNC, CAM3_OUT_BNC, GND, SYNC_IN, SYNC_OUT_INST; removed none
