File: kicad/logic_input_2ch_5v_schmitt_sn74lvc2g17.kicad_sch (KiCad schematic)
At the start: 12 parts, among them U1101 SN74LVC2G17DRYR

Commit message: Regenerate schematics
Parts:
- C1101: Placement (none) -> beside ${d684d2fa-09c2-4534-8acf-a2a601e81a10:REFERENCE}.1 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
- C1102: Placement (none) -> beside ${0c561705-9c07-488f-90ad-207af39ce1e4:REFERENCE}.3 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
- C1103: Placement (none) -> beside ${abd6e6d8-65ef-4922-8cec-490a1d04449e:REFERENCE}.5 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
- R1105: Placement (none) -> beside ${d684d2fa-09c2-4534-8acf-a2a601e81a10:REFERENCE}.6 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
- R1106: Placement (none) -> beside ${0c561705-9c07-488f-90ad-207af39ce1e4:REFERENCE}.4 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
Other:
- note added: "${18be2134-0c6d-468e-977a-6ec186e213ba:REFERENCE} (100 nF) bypasses VCC (pin 5) to GND (pin 2)."
- note added: "${18be2134-0c6d-468e-977a-6ec186e213ba:REFERENCE}: VCC bypass for"
- note added: "${2810be90-e8c8-4226-8b89-017f00ae77cb:REFERENCE}/${b5415b67-1b92-49cb-991a-c122d10e2357:REFERENCE} (100 k) define IN_A/IN_B while the buffer is unpowered;"
- note added: "${2810be90-e8c8-4226-8b89-017f00ae77cb:REFERENCE}/${b5415b67-1b92-49cb-991a-c122d10e2357:REFERENCE} (100 k) define the outputs when +3.3V is off."
- note added: "${2810be90-e8c8-4226-8b89-017f00ae77cb:REFERENCE}: Output pull-down, unpowered state"
- note added: "${485f934b-7a2f-4f64-8b94-d6f4ebd9e779:REFERENCE}/${10c9ffe1-aac2-4e2f-a89b-02c2fadf5966:REFERENCE} (100 ohm) are the series taps to IN_A_INST and IN_B_INST."
- note added: "${504d6ccc-f8c0-42f9-837f-e30ebb7dd752:REFERENCE} in series with the raw input into ${5e0c81c3-f412-4c13-8485-ec7f1d59d7d1:REFERENCE} to GND forms the 72 kHz low-pass at"
- note added: "${5e0c81c3-f412-4c13-8485-ec7f1d59d7d1:REFERENCE}: Input low-pass capacitor, 72 kHz with 4.7 k"
- note added: "${7103dcd1-83f6-4991-a1ac-6565d56e2e67:REFERENCE}: Input low-pass capacitor, 72 kHz with 4.7 k"
- note added: "${99885ad5-2487-4f42-b5fc-c7884fa6dbc3:REFERENCE}/${f3b8ada3-8efc-416a-99a3-6e33fba471fa:REFERENCE} (100 k) pull the raw inputs low when unplugged, on the harness side of the series resistor so no divider eats VIH margin;"
- note added: "${99885ad5-2487-4f42-b5fc-c7884fa6dbc3:REFERENCE}/${f3b8ada3-8efc-416a-99a3-6e33fba471fa:REFERENCE} 100 kohm pull-down (OW-PASS-RC0402JR-07100KL, C106234) on the harness side of the series resistor, so an unplugged input"
- note added: "${abd6e6d8-65ef-4922-8cec-490a1d04449e:REFERENCE} pin 5."
- note added: "${b5415b67-1b92-49cb-991a-c122d10e2357:REFERENCE}: Output pull-down, unpowered state"
- note added: "${d684d2fa-09c2-4534-8acf-a2a601e81a10:REFERENCE}"
- note added: "${d684d2fa-09c2-4534-8acf-a2a601e81a10:REFERENCE} gates A (1A to 1Y) and B (2A to 2Y) square the filtered inputs into 3.3 V logic;"
- note added: "(OW-CAP-470P-0402-C0G-100V, C1518202) and ${d684d2fa-09c2-4534-8acf-a2a601e81a10:REFERENCE} SN74LVC2G17DRYR gate A/B (OW-MISC-SN74LVC2G17DRYR, C2675856);"
- note added: "1. Channel A input filter"
- note added: "1A; ${99885ad5-2487-4f42-b5fc-c7884fa6dbc3:REFERENCE} holds IN_A_RAW low when nothing is plugged in."
- note added: "2. Channel B input filter"
- note added: "3. Output pull-downs and instrument taps"
- note added: "4. Schmitt buffer and supply bypass"
- note added: "Buffer supply (VCC, pin 5), 1.65 to 5.5 V; always-on when the taps must be observable before firmware runs, switched when the consumer of"
- note added: "Conditioned channel A, 3.3 V logic from 1Y (pin 6); pulled down by ${2810be90-e8c8-4226-8b89-017f00ae77cb:REFERENCE} when the rail is off."
- note added: "Conditioned channel B, 3.3 V logic from 2Y (pin 4); pulled down by ${b5415b67-1b92-49cb-991a-c122d10e2357:REFERENCE} when the rail is off."
- note added: "DESIGN CONTRACT"
- note added: "Field-wired channel A input, 0 to 5.5 V legal at any VCC; pulled low by ${99885ad5-2487-4f42-b5fc-c7884fa6dbc3:REFERENCE} (100 k) when unplugged."
- note added: "Field-wired channel B input, 0 to 5.5 V legal at any VCC; pulled low by ${f3b8ada3-8efc-416a-99a3-6e33fba471fa:REFERENCE} (100 k) when unplugged."
- note added: "Filter: 4.7 k and 470 pF give a time constant of about 2.2 us and a corner near 72 kHz; a 3.3 V edge reaches the worst-case VT+ of 2.0 V about 2"
- note added: "Filter: 4.7 kohm and 470 pF give a 72 kHz corner and about 2 us from a 3.3 V edge to the Schmitt threshold, the same on both channels so their"
- note added: "First consumer: camera-gpio-interface-pcb, TRIG IN and SYNC IN BNCs from a pyControl breakout on IN_A_RAW/IN_B_RAW, TRIG_IN/SYNC_IN out, taps"
- note added: "INTERFACES"
- note added: "IN_A/IN_B powers down with it (Ioff keeps the unpowered outputs off the bus)."
- note added: "IN_A_RAW and IN_B_RAW, take conditioned 3.3 V logic out on IN_A and IN_B and the taps out on IN_A_INST and IN_B_INST; rails +3.3V and GND."
- note added: "Input idle-low"
- note added: "Input series filter resistor, 4.7 k"
- note added: "Instrument tap of IN_A through ${485f934b-7a2f-4f64-8b94-d6f4ebd9e779:REFERENCE} (100 ohm), INSTRUMENT class."
- note added: "Instrument tap of IN_B through ${10c9ffe1-aac2-4e2f-a89b-02c2fadf5966:REFERENCE} (100 ohm), INSTRUMENT class."
- note added: "Instrument tap series resistor"
- note added: "Matching net labels are connected. Group order explains function; PCB placement priorities are stated below."
- note added: "OPERATION"
- note added: "PLACE: ${d684d2fa-09c2-4534-8acf-a2a601e81a10:REFERENCE} in the middle of the block between the input and output edges, ${18be2134-0c6d-468e-977a-6ec186e213ba:REFERENCE}"
- note added: "PLACE: Mirror channel A on the input edge so both channels see the same copper and the"
- note added: "PLACE: Output pull-downs and taps on the output edge, so logic and tap nets leave on the"
- note added: "PLACE: Series resistors and filter capacitors on the input edge of the block, ${5e0c81c3-f412-4c13-8485-ec7f1d59d7d1:REFERENCE} with"
- note added: "Per channel: ${504d6ccc-f8c0-42f9-837f-e30ebb7dd752:REFERENCE}/${cd916f99-47ea-446c-b1ea-7b65d79d30fd:REFERENCE} 4.7 kohm series (OW-RES-4K7-0402, C25900) into ${5e0c81c3-f412-4c13-8485-ec7f1d59d7d1:REFERENCE}/${7103dcd1-83f6-4991-a1ac-6565d56e2e67:REFERENCE} 470 pF C0G to ground"
- note added: "Power unit"
- note added: "Project-local pending bench verification; promotable once a second board uses it."
- note added: "ROUTE: +3.3V carries PWR_3V3_LOCAL; the block's baseline is 0.2 mm tracks and 0.6/0.3"
- note added: "ROUTE: IN_A, IN_B, IN_A_INST and IN_B_INST leave through vias (port copper); the taps carry"
- note added: "ROUTE: IN_A_RAW and IN_B_RAW enter as tracks (harness side); IN_A_FILT stays inside the"
- note added: "ROUTE: IN_B_FILT stays inside the block."
- note added: "Rails are generic labels: bind +3.3V to the always-on rail when the taps must be observable before firmware runs, or to the switched domain when"
- note added: "Return for the buffer (pin 2), both filter capacitors and the four pull-downs."
- note added: "Series resistors and filter capacitors on the input edge, the 2G17 and its decoupling in the middle, output pull-downs and taps on the output edge,"
- note added: "Signal path, per channel: IN_A_RAW -> ${504d6ccc-f8c0-42f9-837f-e30ebb7dd752:REFERENCE} (4.7 k) -> IN_A_FILT (${5e0c81c3-f412-4c13-8485-ec7f1d59d7d1:REFERENCE} 470 pF to GND) -> ${d684d2fa-09c2-4534-8acf-a2a601e81a10:REFERENCE} 1A (pin 1) -> 1Y (pin 6) -> IN_A,"
- note added: "Supply: VCC 1.65 to 5.5 V, 10 uA max, +/-24 mA drive at 3 V; Ioff (10 uA max) keeps the outputs off a live downstream input when the rail is down,"
- note added: "The Schmitt input is the point of the block: an ordinary LVC buffer specifies a maximum input transition rate of about 8 ns/V, which a slow or noisy"
- note added: "The Schmitt input is the point: at VCC = 3 V, VT+ is 1.3 to 2.0 V and VT- 0.8 to 1.3 V with at least 0.4 V of hysteresis, so slow or noisy field edges"
- note added: "The same network for channel B into 2A; ${f3b8ada3-8efc-416a-99a3-6e33fba471fa:REFERENCE} holds IN_B_RAW low when unplugged."
- note added: "Tolerance: inputs are rated 0 to 5.5 V at any valid VCC, 6.5 V absolute maximum, with no clamp diode to VCC, so a 5 V source plugged in by mistake"
- note added: "Two-channel Schmitt logic input | 4.7 k / 470 pF filters, SN74LVC2G17, pull-downs and taps"
- note added: "Two-channel single-ended logic input conditioner: per-channel series/RC filtering plus an SN74LVC2G17 dual Schmitt-trigger buffer that turns a 3.3"
- note added: "Two-channel single-ended logic input conditioner: per-channel series/RC filtering plus an SN74LVC2G17 dual Schmitt-trigger buffer that turns a 3.3 V or 5 V field-wired logic signal into clean 3.3 V logic, with a 100 ohm InstrumentPort tap on each output."
- note added: "Unit 1: Schmitt-trigger buffer"
- note added: "Unit 2: Schmitt-trigger buffer"
- note added: "V is bounded to about 7 mA into the buffer."
- note added: "V or 5 V field-wired logic signal into clean 3.3 V logic, with a 100 ohm InstrumentPort tap on each output. Generic sibling of"
- note added: "V, so a 3.3 V microcontroller pin clears the high threshold by 0.9 V or more and a 5 V TTL-level VOH of 2.4 V by 0.4 V."
- note added: "a short return to GND at the buffer's pin 2 side; keep the raw pair away from motor bridge"
- note added: "absolute), so a 5 V source is legal; a source below ground draws about 0.2 mA per volt through the 4.7 k (about 1 mA from -5 V), and a short to 36"
- note added: "block."
- note added: "cannot double-trigger; a 3.3 V source clears VT+ by at least 1.3 V, a 5 V TTL VOH of 2.4 V by 0.4 V. Inputs are rated 0 to 5.5 V at any VCC (6.5 V"
- note added: "disables the outputs when the part is unpowered."
- note added: "downstream buffer never sees a floating input when this rail is down; ${485f934b-7a2f-4f64-8b94-d6f4ebd9e779:REFERENCE}/${10c9ffe1-aac2-4e2f-a89b-02c2fadf5966:REFERENCE} 100 ohm T-taps (OW-PASS-0402WGF1000TCE, C25076) to"
- note added: "encoder supply; place this block twice for four inputs. Connector-agnostic: the jack or terminal lives on the board sheet. Bring the raw lines in on"
- note added: "field edge violates and double-triggers; the 2G17 has no such limit and 0.4 V minimum hysteresis at 3 V. Thresholds VT+ <= 2.0 V and VT- >= 0.8"
- note added: "ground reference."
- note added: "hard against pin 5 with a short return to pin 2; +3.3V and GND reach the block through"
- note added: "is bounded to about 7 mA and destroys a 0.19 USD buffer instead of the consumer."
- note added: "is legal; a source held below ground draws about 0.2 mA per volt through the 4.7 kohm (a -5 V DAC output about 1 mA), and a short to a 36 V rail"
- note added: "mm vias."
- note added: "on DIG0/DIG1 of the digital-50 InstrumentPort."
- note added: "outputs with a ground reference beside it."
- note added: "pull-down, 100 k"
- note added: "quadrature_encoder_input_5v_sn74lvc2g17: same circuit and values, generic names, no encoder-supply passthrough. Use this one for BNC trigger and"
- note added: "reads low without forming a divider that eats VIH margin; ${2810be90-e8c8-4226-8b89-017f00ae77cb:REFERENCE}/${b5415b67-1b92-49cb-991a-c122d10e2357:REFERENCE} 100 kohm pull-down on each output for Ioff high-Z, so an always-on"
- note added: "relative timing is preserved; 470 pF suits sub-10 kHz timing edges on long unshielded leads, swap ${5e0c81c3-f412-4c13-8485-ec7f1d59d7d1:REFERENCE}/${7103dcd1-83f6-4991-a1ac-6565d56e2e67:REFERENCE} for a faster corner when the"
- note added: "same delay."
- note added: "side opposite the harness."
- note added: "signal needs it (27 pF gives 1.25 MHz)."
- note added: "so harness-side nets stay on one edge and logic and tap nets leave on the other. Keep the input pair away from motor bridge outputs and give it a"
- note added: "sync inputs, sensor and switch logic lines and any other pair of inputs a board conditions; use the encoder block when the harness also carries the"
- note added: "tapped through ${485f934b-7a2f-4f64-8b94-d6f4ebd9e779:REFERENCE} (100 ohm) to IN_A_INST; channel B is ${cd916f99-47ea-446c-b1ea-7b65d79d30fd:REFERENCE}, ${7103dcd1-83f6-4991-a1ac-6565d56e2e67:REFERENCE}, 2A (pin 3), 2Y (pin 4), IN_B and ${10c9ffe1-aac2-4e2f-a89b-02c2fadf5966:REFERENCE} to IN_B_INST."
- note added: "the INSTRUMENT class, the two tap stubs are 0.15 mm."
- note added: "the _INST ports, INSTRUMENT netclass from the instrument-taps profile; ${18be2134-0c6d-468e-977a-6ec186e213ba:REFERENCE} 100 nF (OW-CAP-100N-0402-X5R-16V, C162178) hard against"
- note added: "the consumer of IN_A/IN_B can be powered down and must rise and fall with it; sequencing between source and buffer is a non-issue because Ioff"
- note added: "us later, the same on both channels, so relative timing is kept. For faster edges swap ${5e0c81c3-f412-4c13-8485-ec7f1d59d7d1:REFERENCE}/${7103dcd1-83f6-4991-a1ac-6565d56e2e67:REFERENCE} (27 pF gives about 1.25 MHz)."
- note added: "vias."
- note added: "which is why the sequencing between source and buffer does not matter. ${18be2134-0c6d-468e-977a-6ec186e213ba:REFERENCE} (100 nF) bypasses pin 5."
- company: Janelia Research Campus -> Orb Weaver
- title: camera-gpio-interface-pcb -> Two-channel Schmitt logic input
- moved on the sheet: C1101, C1102, C1103, R1101, R1102, R1103, R1104, R1105, R1106, R1107, R1108, U1101A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
