File: kicad/usb2_vertical.kicad_sch (KiCad schematic)
At the start: 6 parts, among them J1 USB-C, U1 USBLC6-2P6

Commit message: Initial v1.0 pcb layout
Parts:
- renumbered C1 to C901, D1 to D901, J1 to J901, R1 to R901, R2 to R902, U1 to U901
Other:
- company: (none) -> Janelia Research Campus
- title: Orb Weaver Design Block Mining -> camera-gpio-interface-pcb
Changed lines of the file:
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@@
 	(paper "A4")
 	(title_block
-		(title "Orb Weaver Design Block Mining")
-		(date "2026-08-28")
+		(title "camera-gpio-interface-pcb")
+		(date "2026-09-25")
+		(rev "1.0")
+		(company "Janelia Research Campus")
 		(comment 1 "Copy or recreate old project circuits here, then save cleaned selections as design blocks.")
 	)
@@
 		(dnp no)
 		(fields_autoplaced yes)
-		(property "Reference" "J1"
+		(property "Reference" "J901"
 			(at 100.33 92.71 0)
 			(show_name no)
@@
 			(project "camera-gpio-interface-pcb"
 				(path "/8c2bf6e9-39ff-46f5-94ad-782f2656bc93/5b8333aa-5632-4b02-bed2-f7f06815639a/891726c4-91ac-4fc5-a699-1590dbecf38b"
-					(reference "J1")
+					(reference "J901")
 					(unit 1)
 				)
@@
 		(in_pos_files yes)
 		(dnp no)
-		(property "Reference" "#FLG01"
+		(property "Reference" "#FLG0901"
 			(at 101.6 38.735 0)
 			(hide yes)
@@
 			(project "camera-gpio-interface-pcb"
 				(path "/8c2bf6e9-39ff-46f5-94ad-782f2656bc93/5b8333aa-5632-4b02-bed2-f7f06815639a/891726c4-91ac-4fc5-a699-1590dbecf38b"
-					(reference "#FLG01")
+					(reference "#FLG0901")
 					(unit 1)
 				)
@@
 		(dnp no)
 		(fields_autoplaced yes)
-		(property "Reference" "C1"
+		(property "Reference" "C901"
 			(at 156.21 63.4999 0)
 			(show_name no)
@@
 			(project "camera-gpio-interface-pcb"
 				(path "/8c2bf6e9-39ff-46f5-94ad-782f2656bc93/5b8333aa-5632-4b02-bed2-f7f06815639a/891726c4-91ac-4fc5-a699-1590dbecf38b"
-					(reference "C1")
+					(reference "C901")
 					(unit 1)
 				)
@@
 		(dnp no)
 		(fields_autoplaced yes)
-		(property "Reference" "D1"
+		(property "Reference" "D901"
 			(at 183.007 57.15 0)
 			(show_name no)
@@
 			(project "camera-gpio-interface-pcb"
 				(path "/8c2bf6e9-39ff-46f5-94ad-782f2656bc93/5b8333aa-5632-4b02-bed2-f7f06815639a/891726c4-91ac-4fc5-a699-1590dbecf38b"
-					(reference "D1")
+					(reference "D901")
 					(unit 1)
 				)
@@
 		(dnp no)
 		(fields_autoplaced yes)
-		(property "Reference" "U1"
+		(property "Reference" "U901"
 			(at 146.4311 86.36 0)
 			(show_name no)
@@
 			(project "camera-gpio-interface-pcb"
 				(path "/8c2bf6e9-39ff-46f5-94ad-782f2656bc93/5b8333aa-5632-4b02-bed2-f7f06815639a/891726c4-91ac-4fc5-a699-1590dbecf38b"
-					(reference "U1")
+					(reference "U901")
 					(unit 1)
 				)
@@
 		(dnp no)
 		(fields_autoplaced yes)
-		(property "Reference" "R1"
+		(property "Reference" "R901"
 			(at 203.2 93.98 0)
 			(show_name no)
@@
 			(project "camera-gpio-interface-pcb"
 				(path "/8c2bf6e9-39ff-46f5-94ad-782f2656bc93/5b8333aa-5632-4b02-bed2-f7f06815639a/891726c4-91ac-4fc5-a699-1590dbecf38b"
-					(reference "R1")
+					(reference "R901")
 					(unit 1)
 				)
@@
 		(dnp no)
 		(fields_autoplaced yes)
-		(property "Reference" "R2"
+		(property "Reference" "R902"
 			(at 218.44 93.98 0)
 			(show_name no)
@@
 			(project "camera-gpio-interface-pcb"
 				(path "/8c2bf6e9-39ff-46f5-94ad-782f2656bc93/5b8333aa-5632-4b02-bed2-f7f06815639a/891726c4-91ac-4fc5-a699-1590dbecf38b"
-					(reference "R2")
+					(reference "R902")
 					(unit 1)
 				)

Commit message: Regenerate schematics
Parts:
- C901, D901: Placement (none) -> beside ${a93e9f9a-5a6f-4043-8a0b-cad9a8361e7e:REFERENCE}.5 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
Connections:
- net USB_D+: now also J901.A6 (D+), J901.B6 (D+), U901.3 (I/O2)
- net USB_D-: now also J901.A7 (D-), J901.B7 (D-), U901.1 (I/O1)
Other:
- note added: "${209f383d-7927-4c04-b30a-21fe2c8eb9bb:REFERENCE} brings VBUS, GND, D+/D-, CC1/CC2 and the shell onto the board; ${a93e9f9a-5a6f-4043-8a0b-cad9a8361e7e:REFERENCE} clamps USB_D+, USB_D- and VBUS to GND right at the receptacle. ${7d317996-fe5e-4d1c-afb9-8653c242779c:REFERENCE} holds the raw VBUS node at"
- note added: "${7d317996-fe5e-4d1c-afb9-8653c242779c:REFERENCE}: VBUS bypass at the clamp"
- note added: "${80f6a5a7-fb59-4c71-91f3-2d3c27fa892a:REFERENCE}: Diode-OR Schottky"
- note added: "${e0574d6f-c3cf-4023-bcca-2b89f01980b8:REFERENCE} and ${e9b764a5-f224-4026-a384-e54737094fce:REFERENCE} (5.1 k) pull CC1 and CC2 to GND: the port presents itself as a sink; nothing reads the source's advertisement."
- note added: "(A1/A12/B1/B12): use all four of each in parallel for the 3 A rating and drop their ties to an inner layer rather than crowding the 1.8 mm corridor"
- note added: "+5V_USB for diode-ORing with other 5 V sources (pair it with pycontrol_behavior_port_rj45's +5V_PYC), PWR_FLAG on VBUS, SBU1/SBU2 deliberately"
- note added: "+5V_USB for diode-ORing with the pyControl block's +5V_PYC. The shell pads S1 to S4 are tied to GND here; isolate them through a pad/cap network"
- note added: "+5V_USB leaves ${80f6a5a7-fb59-4c71-91f3-2d3c27fa892a:REFERENCE} pad 1 into a port via, where a placing board picks the rail up."
- note added: "1. Receptacle and ESD clamp"
- note added: "2. CC sink declaration"
- note added: "3. Power drive declarations"
- note added: "CC Rd sink pulldowns"
- note added: "CC1: Configuration channel for one plug orientation, ${209f383d-7927-4c04-b30a-21fe2c8eb9bb:REFERENCE} A5 to ${e0574d6f-c3cf-4023-bcca-2b89f01980b8:REFERENCE} (Rd, 5.1 k to GND); nothing reads it."
- note added: "CC2: Configuration channel for the other orientation, ${209f383d-7927-4c04-b30a-21fe2c8eb9bb:REFERENCE} B5 to ${e9b764a5-f224-4026-a384-e54737094fce:REFERENCE} (Rd, 5.1 k to GND); nothing reads it."
- note added: "CC: ${e0574d6f-c3cf-4023-bcca-2b89f01980b8:REFERENCE} on CC1 (A5) and ${e9b764a5-f224-4026-a384-e54737094fce:REFERENCE} on CC2 (B5), 5.1 k to GND, declare a UFP (sink). Nothing reads the CC level, so budget the load against a"
- note added: "DESIGN CONTRACT"
- note added: "ESD clamp on D+, D- and VBUS"
- note added: "ESD: ${a93e9f9a-5a6f-4043-8a0b-cad9a8361e7e:REFERENCE} (USBLC6-2P6) clamps D+, D- and VBUS: 3.5 pF max per line, 1.7 pF max line to line, 6 V minimum VBUS breakdown, 12 V typical"
- note added: "INTERFACES"
- note added: "INTERNAL NETS"
- note added: "Keep the USBLC6 hard against the receptacle with a ground via at its pin 2 and route each data line in one I/O pad and out the other (clamp"
- note added: "Land pattern (from the block's own record): contacts in two rows on opposite sides of the body at 0.5 mm pitch, every pad 0.3 mm wide; the A/B ties"
- note added: "Matching net labels are connected. Group order explains function; PCB placement priorities are stated below."
- note added: "Mechanically the courtyard shrinks to x +/-5.05, y +/-2.31 from the horizontal part's x +/-6.00, y -1.25 to +6.75, so the connector stops needing"
- note added: "Nothing reads the CC advertisement, so budget the load against a default-power source unless the host is known to advertise 1.5 A or 3 A."
- note added: "OPERATION"
- note added: "Only the land pattern differs from usb2, and it differs completely, which is why this is a separate block and not a footprint swap: contacts sit in two"
- note added: "PLACE: Keep ${e0574d6f-c3cf-4023-bcca-2b89f01980b8:REFERENCE} at A5 and ${e9b764a5-f224-4026-a384-e54737094fce:REFERENCE} at B5 with short returns; no other load on CC1 or CC2."
- note added: "PLACE: Place ${209f383d-7927-4c04-b30a-21fe2c8eb9bb:REFERENCE}'s four shell-leg holes and two locator pegs before pouring GND or routing the port; the part does not seat without them."
- note added: "PLACE: Place ${7d317996-fe5e-4d1c-afb9-8653c242779c:REFERENCE} between ${a93e9f9a-5a6f-4043-8a0b-cad9a8361e7e:REFERENCE} pin 5 and the GND via; ${80f6a5a7-fb59-4c71-91f3-2d3c27fa892a:REFERENCE} sits where +5V_USB leaves the block at its port via."
- note added: "PLACE: Place ${a93e9f9a-5a6f-4043-8a0b-cad9a8361e7e:REFERENCE} hard against ${209f383d-7927-4c04-b30a-21fe2c8eb9bb:REFERENCE} with a ground via at its pin 2; route each data line in one I/O pad and out the other."
- note added: "Power driven: VBUS"
- note added: "ROUTE: CC1 and CC2 are Default-class local nets that end at the resistors."
- note added: "ROUTE: Jump one leg of each pair once at the body centre for the A/B tie; the 0.3 mm gap at the outer contacts is unroutable."
- note added: "ROUTE: USB_D+ and USB_D- are the USB_HS pair: equal length, coupled at the class gap, brought to the block boundary already coupled."
- note added: "ROUTE: VBUS and +5V_USB are Default-class rails for the port's 5 V budget; +5V_USB is picked up at the port via by the placing board."
- note added: "Raw bus 5 V, ${209f383d-7927-4c04-b30a-21fe2c8eb9bb:REFERENCE} A4, A9, B4, B9; bypassed by ${7d317996-fe5e-4d1c-afb9-8653c242779c:REFERENCE}, the clamp's reference."
- note added: "Signal path: ${209f383d-7927-4c04-b30a-21fe2c8eb9bb:REFERENCE} D+ (A6, B6) and D- (A7, B7) pass ${a93e9f9a-5a6f-4043-8a0b-cad9a8361e7e:REFERENCE}'s I/O pads to USB_D+ and USB_D-; both receptacle rows are tied so either plug"
- note added: "These nets have an explicit ERC power source declaration."
- note added: "USB 2.0 D+, ${209f383d-7927-4c04-b30a-21fe2c8eb9bb:REFERENCE} A6 and B6, after the ${a93e9f9a-5a6f-4043-8a0b-cad9a8361e7e:REFERENCE} clamp; USB_HS pair with USB_D-."
- note added: "USB 2.0 D-, ${209f383d-7927-4c04-b30a-21fe2c8eb9bb:REFERENCE} A7 and B7, after the ${a93e9f9a-5a6f-4043-8a0b-cad9a8361e7e:REFERENCE} clamp; USB_HS pair with USB_D+."
- note added: "USB ground: ${209f383d-7927-4c04-b30a-21fe2c8eb9bb:REFERENCE} A1, B1, A12, B12 and shell S1 to S4; clamp and Rd return."
- note added: "USB-C USB2 device port, vertical receptacle | USB4145, USBLC6 clamp, Rd 5.1 k, 5 V diode-OR"
- note added: "USB-C USB2 device-port front end on a VERTICAL, top-entry receptacle: GCT USB4145-03-0070-C, OW-CONN-USB-C-USB2-SMD-VERT, 16P"
- note added: "USB-C USB2 device-port front end on a VERTICAL, top-entry receptacle: GCT USB4145-03-0070-C, OW-CONN-USB-C-USB2-SMD-VERT, 16P USB2-only, SMT contacts plus four through-hole shell legs, 7.46 mm tall."
- note added: "USB2-only, SMT contacts plus four through-hole shell legs, 7.46 mm tall. Electrically identical to the horizontal usb2 block: USBLC6-2P6 ESD clamp"
- note added: "VBUS through ${80f6a5a7-fb59-4c71-91f3-2d3c27fa892a:REFERENCE} (Schottky, about 0.3 V drop) for diode-ORing with +5V_PYC."
- note added: "VBUS: ${7d317996-fe5e-4d1c-afb9-8653c242779c:REFERENCE} (100 nF) bypasses the raw bus; ${80f6a5a7-fb59-4c71-91f3-2d3c27fa892a:REFERENCE} (MBR120VLSFT1G, 20 V 1 A Schottky, 0.34 V max at 1 A, 0.6 mA leakage at 25 C) makes"
- note added: "about 6.75 mm of board past the contacts and can move inboard, but the cable now leaves perpendicular to the board: the enclosure needs an"
- note added: "aperture above it plus clearance for the plug body and its wire loop, well beyond the 7.46 mm connector height."
- note added: "because the 0.3 mm gap between the outer contact and the shell-leg pad is unroutable at 0.2/0.2 and the plated leg blocks every layer there, so"
- note added: "between the rows, which the two data joins need. The four shell legs are plated ovals on a 1.1 x 0.6 drill at x = +/-4 and punch every layer, and"
- note added: "board (7.46 mm connector height), so the enclosure needs an aperture above it."
- note added: "budget one via jump for one leg of the pair and keep both legs equal length. VBUS lands on four 0.3 mm pads (A4/A9/B4/B9) and GND on four"
- note added: "clamp at 1 A 8/20 us, IEC 61000-4-2 level 4 (15 kV air and contact). Clamp performance is set by connection inductance: pin 2 to a ground via,"
- note added: "default-power source unless the host is known to advertise 1.5 A or 3 A."
- note added: "each data line in one I/O pad and out the other."
- note added: "for D+ and D- cross at the body centre with one via jump per pair leg and equal lengths; VBUS and GND each land on four pads to be used in"
- note added: "for the layout. The A/B ties are the layout's work: D+ (A6/B6) and D- (A7/B7) cross at the body centre and cannot be taken around the ends,"
- note added: "instead if the shield must float."
- note added: "is 0.3 mm wide, where the horizontal GT-USB-7047C merges A and B into one row and gives VBUS and GND 0.6 mm pads. Three consequences follow"
- note added: "on D+/D- and VBUS, 5.1k Rd pulldowns on CC1 (A5) and CC2 (B5) declaring a sink, 100nF on VBUS, a MBR120VLSFT1G series Schottky from VBUS to"
- note added: "orientation works. SBU1 and SBU2 (A8, B8) are no-connect: USB2 only, for an RP2040-class device controller."
- note added: "parallel for the 3 A rating. Four plated shell legs and two 0.71 mm locator pegs are mandatory for seating. The cable leaves perpendicular to the"
- note added: "performance is dominated by connection inductance), and bring USB_D+/USB_D- to the block boundary already coupled at the USB_HS netclass gap."
- note added: "rows on OPPOSITE sides of the body at y = +/-1.485, 0.5 mm pitch across the six inner contacts and 1.5 mm out to the outer pads, and EVERY pad"
- note added: "the clamp; ${80f6a5a7-fb59-4c71-91f3-2d3c27fa892a:REFERENCE} passes VBUS to +5V_USB and blocks the other 5 V source from feeding back into the host."
- note added: "the two 0.71 mm NPTH locator pegs at (+/-4, 0) are mandatory for seating: place all six before pouring GND or routing the port."
- note added: "unconnected, all four shell pads S1-S4 tied to GND. Ports are VBUS, +5V_USB, GND, USB_D+, USB_D-."
- note added: "usb-connector"
- company: Janelia Research Campus -> Orb Weaver
- title: camera-gpio-interface-pcb -> USB-C USB2 device port, vertical
- moved on the sheet: C901, D901, J901, R901, R902, U901
