File: kicad/blackfly_s_gpio_channel_mcv6_vertical.kicad_sch (KiCad schematic)
At the start: 21 parts, among them J701 TBH-1x06-3.5mm, U701 SN74LVC2G17DRYR, U702 SN74LVC1G125DRYR, U703 SN74LVC1G07DRYR, U704 USBLC6-2P6, U705 USBLC6-2P6

Commit message: Regenerate schematics
Parts:
- renumbered C701 to C1401, C702 to C1402, C703 to C1403, D701 to D1401, J701 to J1401, R701 to R1401, R702 to R1402, R703 to R1403, R704 to R1404, R705 to R1405, R706 to R1406, R707 to R1407, R708 to R1408, R709 to R1409, R710 to R1410, R711 to R1411, U701 to U1401, U702 to U1402, U703 to U1403, U704 to U1404, U705 to U1405
Connections:
- net LED_A: now reaches D1401.2 (A), R1406.2
Other:
- note added: "${2227e749-0a2c-4f93-a597-7a23f0e525e1:REFERENCE} pulls Line 2 up, ${e310c8b3-8386-4c71-bde8-59dd025d7495:REFERENCE} gate 1 squares it into CAM_OUT; ${bb6ecb9c-0931-426d-845e-0c0aab3a6240:REFERENCE} drives the BNC, ${7171eb4e-e966-4be1-9b44-87954c581611:REFERENCE} lights ${be5d977c-6c2a-4581-bd66-db9ce884480f:REFERENCE}; ${0eab7050-ae9a-4b12-9155-20dceb5716cb:REFERENCE} pulls Line 1 up and gate 2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"
- note added: "${48a9c958-f5c0-40e3-808a-a90231a7600d:REFERENCE} clamps L3 and L0, ${7159ba13-fb07-4faf-92f2-3f1d229d5679:REFERENCE} clamps L2 and L1, both referenced to +5V and GND; each pair's two I/O pins are tied to the node."
- note added: "${7171eb4e-e966-4be1-9b44-87954c581611:REFERENCE} (680 ohm: about (3.3 - 2.1) / 680 = 1.8 mA, LED on while exposure is active) and the OUT_INST tap. Line 1 (OPTOOUT, LineSource Off) is"
- note added: "${9870f529-44e6-4b20-b7b7-ad6eefe47ea1:REFERENCE}, the 6-position 3.5 mm Phoenix header; pins 1 to 4 are Lines 3, 0, 2 and 1, pins 5 and 6 are the camera's two grounds."
- note added: "${d8715160-be15-46f0-a763-2bd41be97013:REFERENCE} bypasses ${e310c8b3-8386-4c71-bde8-59dd025d7495:REFERENCE}."
- note added: "${dd33be72-e19b-47bb-8c97-5f79fc6338dd:REFERENCE}'s open-drain Y pulls L0 low; ${178e863a-fc0b-474a-a537-37a978202ec6:REFERENCE} (820 ohm) returns it to +5V, the opto input's drive level; ${51f86269-ea15-4394-96b4-401365e1f3d8:REFERENCE} bypasses ${dd33be72-e19b-47bb-8c97-5f79fc6338dd:REFERENCE}'s VCC."
- note added: "${f2a309ed-c3a7-4688-9fba-6e6298bb60c4:REFERENCE} (always enabled) drives L3_DRV; ${e2b2fc18-b9db-4fd9-b2bd-7091a09daaf9:REFERENCE} (220 ohm) in series feeds camera Line 3 on L3; ${10c6213d-5751-476b-ac77-4f982af27ee4:REFERENCE} bypasses ${f2a309ed-c3a7-4688-9fba-6e6298bb60c4:REFERENCE}'s VCC."
- note added: "+3.3V and squared by Schmitt ${e310c8b3-8386-4c71-bde8-59dd025d7495:REFERENCE} 1A -> 1Y = CAM_OUT, which drives the BNC through ${bb6ecb9c-0931-426d-845e-0c0aab3a6240:REFERENCE} (470 ohm), the green LED ${be5d977c-6c2a-4581-bd66-db9ce884480f:REFERENCE} through"
- note added: "+5V, 820 ohm"
- note added: "1 k"
- note added: "1. Camera header"
- note added: "100 ohm series taps: ${36ae1bf1-62f5-4585-a0a5-cbbeae222810:REFERENCE} on L3, ${642b01e2-3cf0-4087-9e79-7690710e4ee1:REFERENCE} on L0, ${c1c7dcbb-7ba6-4d65-abfe-75ca335b5472:REFERENCE} on L2, ${d801cc5a-56c7-46d3-b83c-08021792d765:REFERENCE} on L1_BUF, ${7ee20496-46fb-424b-933f-80f3d28223df:REFERENCE} on CAM_OUT, each to its _INST port."
- note added: "100 ohm tap (${36ae1bf1-62f5-4585-a0a5-cbbeae222810:REFERENCE}) on L3, camera Line 3, the frame trigger."
- note added: "100 ohm tap (${642b01e2-3cf0-4087-9e79-7690710e4ee1:REFERENCE}) on L0, camera Line 0 OPTOIN: the sync drive."
- note added: "100 ohm tap (${7ee20496-46fb-424b-933f-80f3d28223df:REFERENCE}) on CAM_OUT, the buffered exposure signal."
- note added: "100 ohm tap (${c1c7dcbb-7ba6-4d65-abfe-75ca335b5472:REFERENCE}) on L2, camera Line 2, the open-drain exposure output."
- note added: "100 ohm tap (${d801cc5a-56c7-46d3-b83c-08021792d765:REFERENCE}) on L1_BUF, camera Line 1 OPTOOUT after the Schmitt buffer."
- note added: "100 ohm tap, CAM_OUT to OUT_INST"
- note added: "100 ohm tap, L0 to L0_INST"
- note added: "100 ohm tap, L1_BUF to L1_INST"
- note added: "100 ohm tap, L2 to L2_INST"
- note added: "100 ohm tap, L3 to L3_INST"
- note added: "2. Line 3 trigger drive"
- note added: "3. Line 0 sync drive"
- note added: "3.5 mm"
- note added: "3.5 mm, origin at the pad-array centre), so the variant swaps only the connector's body, courtyard and 3D model; every pad, track and via stays, and"
- note added: "4 white Line 1 (OPTOOUT), pin 5 blue opto ground and pin 6 brown ground, both on GND (common-ground wiring)."
- note added: "4. Exposure output, BNC drive and LED"
- note added: "4.7 k"
- note added: "5. ESD clamps"
- note added: "5.5 V-tolerant I/O."
- note added: "6. Instrument taps"
- note added: "BNC drive series, 470 ohm"
- note added: "Blackfly S GPIO channel | trigger in, sync in, exposure out, five taps; vertical or horizontal header"
- note added: "CAM_OUT: Buffered Line 2 (exposure active) from ${e310c8b3-8386-4c71-bde8-59dd025d7495:REFERENCE} 1Y; drives the BNC resistor, the LED resistor and the OUT tap."
- note added: "Camera GPIO header, 6-pos"
- note added: "Camera pins 5 (opto ground) and 6 (ground) both land here, with the logic and ESD returns."
- note added: "Camera side: ${9870f529-44e6-4b20-b7b7-ad6eefe47ea1:REFERENCE}'s terminal numbers are the camera's Hirose HR10A-7R-6PB pin numbers, wired with the FLIR 1 m flying-lead GPIO cable into"
- note added: "Conditioned 3.3 V Rsync from the board's input Schmitt into ${dd33be72-e19b-47bb-8c97-5f79fc6338dd:REFERENCE} (pin 2)."
- note added: "Conditioned 3.3 V frame trigger from the board's input Schmitt into ${f2a309ed-c3a7-4688-9fba-6e6298bb60c4:REFERENCE} (pin 2)."
- note added: "DESIGN CONTRACT"
- note added: "ESD array for L2/L1"
- note added: "ESD array for L3/L0"
- note added: "ESD: two USBLC6-2P6 arrays with VBUS on +5V clamp L3 and L0 (${48a9c958-f5c0-40e3-808a-a90231a7600d:REFERENCE}) and L2 and L1 (${7159ba13-fb07-4faf-92f2-3f1d229d5679:REFERENCE}), 15 kV IEC 61000-4-2 level 4, at most 3.5"
- note added: "Exposure LED, green"
- note added: "Exposure output: camera Line 2 (LineMode Output, LineSource ExposureActive, V3_3Enable false, so open drain) is pulled up by ${2227e749-0a2c-4f93-a597-7a23f0e525e1:REFERENCE} (1 k) to"
- note added: "Exposure-active output: CAM_OUT through ${bb6ecb9c-0931-426d-845e-0c0aab3a6240:REFERENCE} (470 ohm); the BNC itself is the board's."
- note added: "INTERFACES"
- note added: "INTERNAL NETS"
- note added: "L0 opto pull-up to"
- note added: "L0, pulled to +5V by ${178e863a-fc0b-474a-a537-37a978202ec6:REFERENCE} (820 ohm): 5 V across 820 ohm is about 6 mA, less by the opto input's forward drop. Both drivers run from +3.3V with"
- note added: "L0: Camera pin 2, Line 0 OPTOIN: open-drain ${dd33be72-e19b-47bb-8c97-5f79fc6338dd:REFERENCE} Y, pulled to +5V by ${178e863a-fc0b-474a-a537-37a978202ec6:REFERENCE} (820 ohm), clamped by ${48a9c958-f5c0-40e3-808a-a90231a7600d:REFERENCE}."
- note added: "L1 pull-up to +3.3V,"
- note added: "L1: Camera pin 4, Line 1 OPTOOUT, pulled up to +3.3V by ${0eab7050-ae9a-4b12-9155-20dceb5716cb:REFERENCE} (4.7 k), into Schmitt 2A, clamped by ${7159ba13-fb07-4faf-92f2-3f1d229d5679:REFERENCE}."
- note added: "L1_BUF: Schmitt 2Y: buffered Line 1 for the L1_INST tap."
- note added: "L2 pull-up to +3.3V,"
- note added: "L2: Camera pin 3, Line 2 as open-drain exposure output, pulled up by ${2227e749-0a2c-4f93-a597-7a23f0e525e1:REFERENCE} (1 k), into Schmitt 1A, clamped by ${7159ba13-fb07-4faf-92f2-3f1d229d5679:REFERENCE}."
- note added: "L3 trigger series, 220 ohm"
- note added: "L3: Camera pin 1, Line 3 GPI trigger, driven by ${f2a309ed-c3a7-4688-9fba-6e6298bb60c4:REFERENCE} through ${e2b2fc18-b9db-4fd9-b2bd-7091a09daaf9:REFERENCE} (220 ohm), clamped by ${48a9c958-f5c0-40e3-808a-a90231a7600d:REFERENCE}."
- note added: "L3_DRV: ${f2a309ed-c3a7-4688-9fba-6e6298bb60c4:REFERENCE} Y, the trigger drive before the 220 ohm series resistor."
- note added: "LED series, 680 ohm"
- note added: "LED_A: LED anode: ${7171eb4e-e966-4be1-9b44-87954c581611:REFERENCE} (680 ohm) from CAM_OUT, so ${be5d977c-6c2a-4581-bd66-db9ce884480f:REFERENCE} lights while exposure is active."
- note added: "Line 0 sync driver, open drain"
- note added: "Line 3 trigger driver, always enabled"
- note added: "Line 3; camera settings TriggerSelector FrameStart, TriggerSource Line3 RisingEdge. Sync path: SYNC_IN -> ${dd33be72-e19b-47bb-8c97-5f79fc6338dd:REFERENCE} (SN74LVC1G07 open drain) ->"
- note added: "Logic rail for ${e310c8b3-8386-4c71-bde8-59dd025d7495:REFERENCE}, ${f2a309ed-c3a7-4688-9fba-6e6298bb60c4:REFERENCE}, ${dd33be72-e19b-47bb-8c97-5f79fc6338dd:REFERENCE} and the L2/L1 pull-ups; always-on if the taps must read before firmware."
- note added: "Matching net labels are connected. Group order explains function; PCB placement priorities are stated below."
- note added: "Must be a 5 V rail: the Line 0 opto drive level (${178e863a-fc0b-474a-a537-37a978202ec6:REFERENCE}) and both ESD clamps' VBUS reference."
- note added: "OPERATION"
- note added: "OW-CONN-1844252 (Phoenix MC 1,5/6-G-3,5, side entry toward the footprint's +Y). The two footprints are pad-identical (six 1.8 x 3.6 mm ovals on"
- note added: "One FLIR Blackfly S camera GPIO channel (trigger, sync, exposure output, instrument taps) on a 6-position 3.5 mm Phoenix header; the connector"
- note added: "One FLIR Blackfly S camera GPIO channel (trigger, sync, exposure output, instrument taps) on a 6-position 3.5 mm Phoenix header; the connector family pilot: the vertical MCV and the horizontal MC header are pad-identical, so one source publishes both orientations"
- note added: "PLACE: Place ${9870f529-44e6-4b20-b7b7-ad6eefe47ea1:REFERENCE} at the board edge the plug needs: the vertical body takes the plug from above, the horizontal from its +Y side; the anchor is the pad-array centre for both."
- note added: "PLACE: Place ${dd33be72-e19b-47bb-8c97-5f79fc6338dd:REFERENCE} near ${9870f529-44e6-4b20-b7b7-ad6eefe47ea1:REFERENCE} pin 2 with ${51f86269-ea15-4394-96b4-401365e1f3d8:REFERENCE} at its pin 6; ${178e863a-fc0b-474a-a537-37a978202ec6:REFERENCE} from L0 to the +5V entry."
- note added: "PLACE: Place ${e310c8b3-8386-4c71-bde8-59dd025d7495:REFERENCE} between the connector and the BNC side with ${d8715160-be15-46f0-a763-2bd41be97013:REFERENCE} at its pin 5; ${2227e749-0a2c-4f93-a597-7a23f0e525e1:REFERENCE} and ${0eab7050-ae9a-4b12-9155-20dceb5716cb:REFERENCE} at the connector pads; ${be5d977c-6c2a-4581-bd66-db9ce884480f:REFERENCE} where it is visible."
- note added: "PLACE: Place ${f2a309ed-c3a7-4688-9fba-6e6298bb60c4:REFERENCE} near ${9870f529-44e6-4b20-b7b7-ad6eefe47ea1:REFERENCE} pin 1 with ${10c6213d-5751-476b-ac77-4f982af27ee4:REFERENCE} at its pin 6 and a short return to pin 3; ${e2b2fc18-b9db-4fd9-b2bd-7091a09daaf9:REFERENCE} between the driver and the connector."
- note added: "PLACE: Place both arrays right at ${9870f529-44e6-4b20-b7b7-ad6eefe47ea1:REFERENCE}'s pads, before any series part, with the shortest GND return."
- note added: "PLACE: Place the five taps as a row toward the instrument-port side of the block."
- note added: "Power unit"
- note added: "ROUTE: CAM_OUT is the board's exposure reference: route ${bb6ecb9c-0931-426d-845e-0c0aab3a6240:REFERENCE}'s far end to the BNC with a ground return beside it."
- note added: "ROUTE: INSTRUMENT class to the instrument port; every tapped node has a DC definition (driven or pulled up)."
- note added: "ROUTE: L0 carries about 6 mA pulses into the camera's opto input; keep its return with the trigger line."
- note added: "ROUTE: L3 is a 3.3 V edge-triggered line: short, over ground, away from the switching parts of the board."
- note added: "ROUTE: L3, L0, L2 and L1 run straight from the pads to their clamps and parts; GND from pins 5 and 6 into the block's return."
- note added: "ROUTE: Wire the paired I/O pads together on the node itself; no separate track between them."
- note added: "The placing board provides +3.3V (bind it to the always-on rail when the taps must be observable before firmware runs), a 5 V rail on +5V, the BNC"
- note added: "Trigger path: TRIG_IN -> ${f2a309ed-c3a7-4688-9fba-6e6298bb60c4:REFERENCE} (SN74LVC1G125, ~{OE} pin 1 grounded, so always enabled) -> L3_DRV -> ${e2b2fc18-b9db-4fd9-b2bd-7091a09daaf9:REFERENCE} (220 ohm) -> L3 -> camera"
- note added: "Unit 1: Schmitt buffers, L2 and L1"
- note added: "Unit 2: Schmitt buffers, L2 and L1"
- note added: "V rail: it is the clamp reference and the opto drive level, and feeds nothing else."
- note added: "VCC pin 5 bypass, ${e310c8b3-8386-4c71-bde8-59dd025d7495:REFERENCE}"
- note added: "VCC pin 6 bypass, ${dd33be72-e19b-47bb-8c97-5f79fc6338dd:REFERENCE}"
- note added: "VCC pin 6 bypass, ${f2a309ed-c3a7-4688-9fba-6e6298bb60c4:REFERENCE}"
- note added: "Variants (family.json): mcv6_vertical fits ${9870f529-44e6-4b20-b7b7-ad6eefe47ea1:REFERENCE} = OW-CONN-TBH-1X06-3P5-VERT (Phoenix MCV 1,5/6-G-3,5, top entry); mc6_horizontal fits"
- note added: "a Phoenix MC 1,5/6-ST-3,5 plug: pin 1 green Line 3 (GPI, trigger), pin 2 black Line 0 (OPTOIN, sync), pin 3 red Line 2 (GPIO, exposure output), pin"
- note added: "because the block owns L0, L1 and L2 (layout convention 10). Place one block per camera; the horizontal variant's plug needs the board edge its wire"
- note added: "exit faces."
- note added: "family pilot: the vertical MCV and the horizontal MC header are pad-identical, so one source publishes both orientations"
- note added: "on CAM_OUT_BNC, the conditioned 3.3 V TRIG_IN and SYNC_IN, and the instrument port behind the five 100 ohm taps; the three pull-ups are inside"
- note added: "pF per line; both I/O pins of each pair are wired to the node, so the footprint's paired pads need no track between them. +5V must therefore be a 5"
- note added: "pulled up by ${0eab7050-ae9a-4b12-9155-20dceb5716cb:REFERENCE} (4.7 k) and buffered 2A -> 2Y into L1_BUF for its tap."
- note added: "the anchor connector_center is the same point for both."
- company: Janelia Research Campus -> Orb Weaver
- title: camera-gpio-interface-pcb -> Blackfly S GPIO channel family
- moved on the sheet: C1401, C1402, C1403, D1401, J1401, R1401, R1402, R1403, R1404, R1405, R1406, R1407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

Commit message: Regenerate schematics
Parts:
- C1201: renamed from C1401; Placement (none) -> beside ${f2a309ed-c3a7-4688-9fba-6e6298bb60c4:REFERENCE}.6 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
- C1202: renamed from C1402; Placement (none) -> beside ${dd33be72-e19b-47bb-8c97-5f79fc6338dd:REFERENCE}.6 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
- C1203: renamed from C1403; Placement (none) -> beside ${7b072c8a-4743-483b-985c-6774fd37fcc8:REFERENCE}.5 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
- R1201: renamed from R1401; Placement (none) -> beside ${e310c8b3-8386-4c71-bde8-59dd025d7495:REFERENCE}.1 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
- R1202: renamed from R1402; Placement (none) -> beside ${f6b885c6-bea8-4f63-a8bf-ed54c18ce440:REFERENCE}.3 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
- R1203: renamed from R1403; Placement (none) -> beside ${dd33be72-e19b-47bb-8c97-5f79fc6338dd:REFERENCE}.4,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
- renumbered D1401 to D1201, J1401 to J1201, R1404 to R1204, R1405 to R1205, R1406 to R1206, R1407 to R1207, R1408 to R1208, R1409 to R1209, R1410 to R1210, R1411 to R1211, U1401 to U1201, U1402 to U1202, U1403 to U1203, U1404 to U1204, U1405 to U1205
