File: kicad/instrument_port_digital_50_dut_ffc_boundary_vertical.kicad_sch (KiCad schematic)
At the start: 46 parts, among them J501 FH12-50S-0.5SVA(54), U501 SN74LV541ARKSR, U502 SN74LV541ARKSR, U503 SN74LV541ARKSR, U504 SN74LV541ARKSR

Commit message: Regenerate schematics
Other:
- note added: "${27c0d602-bef6-4707-9c9a-9a3c429a569d:REFERENCE} carries the 32 damped outputs (DIGn_ISO) on the contract's DUT contacts and the 18 grounds on one GND; the four mechanical lands carry no net."
- note added: "${32c854d3-e295-4ed0-ae67-c404202c33c2:REFERENCE} bypasses VCC (pin 20); ${84c143f8-b8f7-412f-b388-3f55d62abdd6:REFERENCE} holds both enables (pins 1 and 19) low."
- note added: "${3b73245c-fad3-495c-87fd-b301079bbe35:REFERENCE} (4.7 uF) holds the +3.3V rail where it enters the block; the per-package 100 nF bypasses are in the octet groups."
- note added: "${69119102-0ebd-473d-a7cb-d952bc88de42:REFERENCE} buffers DIG16 to DIG23 (inputs A8 to A1, pins 9 to 2) onto Y8 to Y1 (pins 11 to 18); ${12aa9e00-ffcb-4158-821b-7de5cab15da1:REFERENCE} to ${afc42ada-6ba1-45cb-a7b0-fa0300973df2:REFERENCE} (100 ohm) damp each output into its connector contact."
- note added: "${7e0cdabf-d9e1-4b13-ab00-5a4417fdb564:REFERENCE} buffers DIG0 to DIG7 (inputs A8 to A1, pins 9 to 2) onto Y8 to Y1 (pins 11 to 18); ${fad54bc1-8b2f-4c3f-a18e-9b2430ab141a:REFERENCE} to ${fcea49a0-ea4d-4aee-9697-0faa5db34934:REFERENCE} (100 ohm) damp each output into its connector contact."
- note added: "${889f984f-3f59-44b0-b31b-4ed72ef307ca:REFERENCE} bypasses VCC (pin 20); ${b78c2658-d37d-41d9-a37f-c55fb33c8270:REFERENCE} holds both enables (pins 1 and 19) low."
- note added: "${97871112-ad18-45a1-a62c-deaacd916849:REFERENCE} bypasses VCC (pin 20); ${6c63e654-1b93-4601-99a7-45c9ca25760f:REFERENCE} holds both enables (pins 1 and 19) low."
- note added: "${b1707ec3-0f6f-4e89-a1c4-65233bece57d:REFERENCE} buffers DIG8 to DIG15 (inputs A8 to A1, pins 9 to 2) onto Y8 to Y1 (pins 11 to 18); ${e1d059cd-edbc-42a0-8ffd-62ba15148778:REFERENCE} to ${bbf3e143-2a2a-405b-bcb8-81ea8fc164d3:REFERENCE} (100 ohm) damp each output into its connector contact."
- note added: "${f13cd1d5-28c7-4506-b50d-dbf0bfbd6248:REFERENCE} buffers DIG24 to DIG31 (inputs A8 to A1, pins 9 to 2) onto Y8 to Y1 (pins 11 to 18); ${7850a50d-bc57-46a0-9379-26c0e7edf3c1:REFERENCE} to ${b42723d6-d7f2-4621-8097-95df4034dcaa:REFERENCE} (100 ohm) damp each output into its connector contact."
- note added: "${fbe8828a-42e9-430d-9de7-defb4cc837f2:REFERENCE} bypasses VCC (pin 20); ${a0f1ba57-587e-4049-9916-5b2de5f5036d:REFERENCE} holds both enables (pins 1 and 19) low."
- note added: "(DIG0 to 7, 8 to 15, 16 to 23, 24 to 31, each octet one package, A8 down to A1), leaves on Y8 to Y1 through 100 ohm damping (${fad54bc1-8b2f-4c3f-a18e-9b2430ab141a:REFERENCE} to ${b42723d6-d7f2-4621-8097-95df4034dcaa:REFERENCE}) onto ${27c0d602-bef6-4707-9c9a-9a3c429a569d:REFERENCE}. The cable carries no supply,"
- note added: "+3.3V rail-entry bulk,"
- note added: "1. Octet DIG0 to DIG7: ${7e0cdabf-d9e1-4b13-ab00-5a4417fdb564:REFERENCE}"
- note added: "10 k"
- note added: "18 connector grounds, buffer GND pins and pads, bypass and OE pull-down return."
- note added: "2. Octet DIG8 to DIG15: ${b1707ec3-0f6f-4e89-a1c4-65233bece57d:REFERENCE}"
- note added: "3. Octet DIG16 to DIG23: ${69119102-0ebd-473d-a7cb-d952bc88de42:REFERENCE}"
- note added: "4. Octet DIG24 to DIG31: ${f13cd1d5-28c7-4506-b50d-dbf0bfbd6248:REFERENCE}"
- note added: "4.7 uF"
- note added: "5. Rail-entry bulk bypass"
- note added: "50-contact FFC receptacle, top entry"
- note added: "541 is flow-through: input pin p pairs with output pin 20-p, A1(2) to Y1(18) through A8(9) to Y8(11). DIRECTION IS A HARDWARE PROPERTY: DUT to instrument only. The cable carries no supply, no voltage"
- note added: "6. FFC receptacle"
- note added: "Always-on 3.3 V buffer supply (VCC pins 20); never reaches the cable."
- note added: "C597991, 0.5mm pitch, symbol Conn_01x50, footprint orb_weaver_connectors:Hirose_FH12-50S-0.5SVA_1x50-4MP_P0.5mm_Vertical; the four mechanical lands are unnumbered pads and carry no net."
- note added: "DESIGN CONTRACT"
- note added: "DUT side of the InstrumentPort-Digital-50 profile (board-interfaces docs/instrument-port-digital.md, draft v0.1). Direction is a hardware property, DUT to instrument only: DIGn enters ${7e0cdabf-d9e1-4b13-ab00-5a4417fdb564:REFERENCE} to ${f13cd1d5-28c7-4506-b50d-dbf0bfbd6248:REFERENCE}"
- note added: "DUT-side InstrumentPort-Digital-50 with integrated read-only buffering, on a VERTICAL, top-entry 50-contact ZIF connector: Hirose FH12-50S-0.5SVA(54), OW-CONN-FH12-50S-0-5SVA-54, LCSC"
- note added: "DUT-side InstrumentPort-Digital-50 with integrated read-only buffering, on a VERTICAL, top-entry 50-contact ZIF connector: Hirose FH12-50S-0.5SVA(54), OW-CONN-FH12-50S-0-5SVA-54, LCSC C597991, 0.5mm pitch, symbol Conn_01x50, footprint orb_weaver_connectors:Hirose_FH12-50S-0.5SVA_1x50-4MP_P0.5mm_Vertical; the four mechanical lands are unnumbered pads and carry no net."
- note added: "Enabled by hardware default, no disable at all: both active-low enables of each package share one net held low by its 10 k pull-down (${84c143f8-b8f7-412f-b388-3f55d62abdd6:REFERENCE} to ${6c63e654-1b93-4601-99a7-45c9ca25760f:REFERENCE}; at most about 0.1 V from the two inputs'"
- note added: "INTERFACES"
- note added: "InstrumentPort-Digital-50 DUT boundary | four SN74LV541A octets, 100 ohm damping, enabled by hardware"
- note added: "Marker/beacon channel indices are NOT frozen, with DIG0/DIG1 the current recommendation over the earlier DIG14/DIG15. Pairs with instrument_port_digital_50_adapter_ffc_boundary_vertical; the"
- note added: "Matching net labels are connected. Group order explains function; PCB placement priorities are stated below."
- note added: "NOT HERE. instrument_port_digital_50_adapter_ffc_boundary_vertical is pre-mirrored to 51-n so that the expected reversing assembly - same-side Type A FFC with a vertical FH12 at both ends, connectors"
- note added: "OPERATION"
- note added: "Observation input 0 into ${7e0cdabf-d9e1-4b13-ab00-5a4417fdb564:REFERENCE} A8 (pin 9); leaves on contact 2."
- note added: "Observation input 1 into ${7e0cdabf-d9e1-4b13-ab00-5a4417fdb564:REFERENCE} A7 (pin 8); leaves on contact 3."
- note added: "Observation input 10 into ${b1707ec3-0f6f-4e89-a1c4-65233bece57d:REFERENCE} A6 (pin 7); leaves on contact 17."
- note added: "Observation input 11 into ${b1707ec3-0f6f-4e89-a1c4-65233bece57d:REFERENCE} A5 (pin 6); leaves on contact 18."
- note added: "Observation input 12 into ${b1707ec3-0f6f-4e89-a1c4-65233bece57d:REFERENCE} A4 (pin 5); leaves on contact 20."
- note added: "Observation input 13 into ${b1707ec3-0f6f-4e89-a1c4-65233bece57d:REFERENCE} A3 (pin 4); leaves on contact 21."
- note added: "Observation input 14 into ${b1707ec3-0f6f-4e89-a1c4-65233bece57d:REFERENCE} A2 (pin 3); leaves on contact 23."
- note added: "Observation input 15 into ${b1707ec3-0f6f-4e89-a1c4-65233bece57d:REFERENCE} A1 (pin 2); leaves on contact 24."
- note added: "Observation input 16 into ${69119102-0ebd-473d-a7cb-d952bc88de42:REFERENCE} A8 (pin 9); leaves on contact 27."
- note added: "Observation input 17 into ${69119102-0ebd-473d-a7cb-d952bc88de42:REFERENCE} A7 (pin 8); leaves on contact 28."
- note added: "Observation input 18 into ${69119102-0ebd-473d-a7cb-d952bc88de42:REFERENCE} A6 (pin 7); leaves on contact 30."
- note added: "Observation input 19 into ${69119102-0ebd-473d-a7cb-d952bc88de42:REFERENCE} A5 (pin 6); leaves on contact 31."
- note added: "Observation input 2 into ${7e0cdabf-d9e1-4b13-ab00-5a4417fdb564:REFERENCE} A6 (pin 7); leaves on contact 5."
- note added: "Observation input 20 into ${69119102-0ebd-473d-a7cb-d952bc88de42:REFERENCE} A4 (pin 5); leaves on contact 33."
- note added: "Observation input 21 into ${69119102-0ebd-473d-a7cb-d952bc88de42:REFERENCE} A3 (pin 4); leaves on contact 34."
- note added: "Observation input 22 into ${69119102-0ebd-473d-a7cb-d952bc88de42:REFERENCE} A2 (pin 3); leaves on contact 36."
- note added: "Observation input 23 into ${69119102-0ebd-473d-a7cb-d952bc88de42:REFERENCE} A1 (pin 2); leaves on contact 37."
- note added: "Observation input 24 into ${f13cd1d5-28c7-4506-b50d-dbf0bfbd6248:REFERENCE} A8 (pin 9); leaves on contact 39."
- note added: "Observation input 25 into ${f13cd1d5-28c7-4506-b50d-dbf0bfbd6248:REFERENCE} A7 (pin 8); leaves on contact 40."
- note added: "Observation input 26 into ${f13cd1d5-28c7-4506-b50d-dbf0bfbd6248:REFERENCE} A6 (pin 7); leaves on contact 42."
- note added: "Observation input 27 into ${f13cd1d5-28c7-4506-b50d-dbf0bfbd6248:REFERENCE} A5 (pin 6); leaves on contact 43."
- note added: "Observation input 28 into ${f13cd1d5-28c7-4506-b50d-dbf0bfbd6248:REFERENCE} A4 (pin 5); leaves on contact 45."
- note added: "Observation input 29 into ${f13cd1d5-28c7-4506-b50d-dbf0bfbd6248:REFERENCE} A3 (pin 4); leaves on contact 46."
- note added: "Observation input 3 into ${7e0cdabf-d9e1-4b13-ab00-5a4417fdb564:REFERENCE} A5 (pin 6); leaves on contact 6."
- note added: "Observation input 30 into ${f13cd1d5-28c7-4506-b50d-dbf0bfbd6248:REFERENCE} A2 (pin 3); leaves on contact 48."
- note added: "Observation input 31 into ${f13cd1d5-28c7-4506-b50d-dbf0bfbd6248:REFERENCE} A1 (pin 2); leaves on contact 49."
- note added: "Observation input 4 into ${7e0cdabf-d9e1-4b13-ab00-5a4417fdb564:REFERENCE} A4 (pin 5); leaves on contact 8."
- note added: "Observation input 5 into ${7e0cdabf-d9e1-4b13-ab00-5a4417fdb564:REFERENCE} A3 (pin 4); leaves on contact 9."
- note added: "Observation input 6 into ${7e0cdabf-d9e1-4b13-ab00-5a4417fdb564:REFERENCE} A2 (pin 3); leaves on contact 11."
- note added: "Observation input 7 into ${7e0cdabf-d9e1-4b13-ab00-5a4417fdb564:REFERENCE} A1 (pin 2); leaves on contact 12."
- note added: "Observation input 8 into ${b1707ec3-0f6f-4e89-a1c4-65233bece57d:REFERENCE} A8 (pin 9); leaves on contact 14."
- note added: "Observation input 9 into ${b1707ec3-0f6f-4e89-a1c4-65233bece57d:REFERENCE} A7 (pin 8); leaves on contact 15."
- note added: "Output source damping"
- note added: "PLACE: Place ${32c854d3-e295-4ed0-ae67-c404202c33c2:REFERENCE} hard against pin 20 of ${7e0cdabf-d9e1-4b13-ab00-5a4417fdb564:REFERENCE} with a short return to pin 10 and the exposed pad 21; ${84c143f8-b8f7-412f-b388-3f55d62abdd6:REFERENCE} near pins 1 and 19; the eight damping resistors"
- note added: "PLACE: Place ${3b73245c-fad3-495c-87fd-b301079bbe35:REFERENCE} at the supply entry of the block, not at any one package."
- note added: "PLACE: Place ${889f984f-3f59-44b0-b31b-4ed72ef307ca:REFERENCE} hard against pin 20 of ${b1707ec3-0f6f-4e89-a1c4-65233bece57d:REFERENCE} with a short return to pin 10 and the exposed pad 21; ${b78c2658-d37d-41d9-a37f-c55fb33c8270:REFERENCE} near pins 1 and 19; the eight damping resistors"
- note added: "PLACE: Place ${97871112-ad18-45a1-a62c-deaacd916849:REFERENCE} hard against pin 20 of ${f13cd1d5-28c7-4506-b50d-dbf0bfbd6248:REFERENCE} with a short return to pin 10 and the exposed pad 21; ${6c63e654-1b93-4601-99a7-45c9ca25760f:REFERENCE} near pins 1 and 19; the eight damping resistors"
- note added: "PLACE: Place ${fbe8828a-42e9-430d-9de7-defb4cc837f2:REFERENCE} hard against pin 20 of ${69119102-0ebd-473d-a7cb-d952bc88de42:REFERENCE} with a short return to pin 10 and the exposed pad 21; ${a0f1ba57-587e-4049-9916-5b2de5f5036d:REFERENCE} near pins 1 and 19; the eight damping resistors"
- note added: "PLACE: Vertical, top-entry receptacle at the board edge, latch away from the buffers; verify pin 1 and the contact face on the real part."
- note added: "Per-output source damping is 100 ohms, OW-PASS-0402WGF1000TCE. That value is chosen as the smallest standard one that bounds a hard short to ground inside the LV541A's +/-35mA output absolute"
- note added: "Pin mapping is the contract's DUT table and is not mirrored: channel n lands on contact 2 + n + floor(n/2) + floor(n/16), DIG0 on contact 2, DIG31 on contact 49, the 18 grounds on 1, 4, 7, ... 47, 50"
- note added: "ROUTE: +3.3V carries PWR_3V3_LOCAL from the entry to the four VCC pins; GND is PWR_RETURN_LOCAL."
- note added: "ROUTE: Pair each DIGn_ISO with its neighbouring ground contact and tie all 18 grounds into one GND copper under the connector; land pattern dual-row staggered at 1.0 mm"
- note added: "ROUTE: The DIG0 to DIG7 inputs are this block's ports and escape toward the board on vias; keep the Y runs short to the resistors and the resistor-to-contact runs paired"
- note added: "ROUTE: The DIG16 to DIG23 inputs are this block's ports and escape toward the board on vias; keep the Y runs short to the resistors and the resistor-to-contact runs paired"
- note added: "ROUTE: The DIG24 to DIG31 inputs are this block's ports and escape toward the board on vias; keep the Y runs short to the resistors and the resistor-to-contact runs paired"
- note added: "ROUTE: The DIG8 to DIG15 inputs are this block's ports and escape toward the board on vias; keep the Y runs short to the resistors and the resistor-to-contact runs paired"
- note added: "SN74LV541A octal buffer, DUT to instrument"
- note added: "Supply: the always-on 3.3 V rail on VCC (pins 20); SN74LV541A runs 2 to 5.5 V, drives +/-8 mA at 3.3 V, inputs tolerate 0 to 5.5 V with Ioff <= 5 uA unpowered, VIH 2.31 V, VIL 0.99 V, edges <= 100"
- note added: "The 100 ohm damping bounds a hard short of one output to GND at 33 mA, inside the +/-35 mA per-output absolute maximum, and damps edges into the cable; it is not short-circuit protection. Input"
- note added: "Thirty-two channels through four SN74LV541ARKSR octal buffers (OW-MISC-SN74LV541ARKSR, C7364695, symbol orb_weaver_misc:SN74LV541ARKSR, footprint"
- note added: "VCC pin 20 bypass, 100 nF"
- note added: "analyzer-specific channel map belongs to la5032_connector_boundary, not here. GROUNDED INPUTS ARE THE BOARD'S COPPER: the inputs are this block's ports, so a board that grounds unused DIGn"
- note added: "and damping resistors; lift the 100R resistors on the suspect channels instead. SUPPLY FROM THE BOARD'S ALWAYS-ON 3.3V RAIL, independent of firmware, HV_EN and every switched domain; a buffer on a"
- note added: "and every net stays driven and terminated: ERC, DRC and design_block_tools.py check are ALL BLIND to this error, and only a pin-by-pin netlist comparison or continuity on the real cable catches it."
- note added: "and the LV541A pins (2026-09-26) and between each DIGn escape stub and the escape via beside it (2026-09-29) are wrapped in BLOCK_FLOOR rule areas, so a consuming board sees no clearance"
- note added: "between the Y pins and ${27c0d602-bef6-4707-9c9a-9a3c429a569d:REFERENCE}, outputs toward the connector."
- note added: "bias is board-specific and not in this block: every unused DIGn must be tied at the board. Attach and remove the FFC with target power off; ${27c0d602-bef6-4707-9c9a-9a3c429a569d:REFERENCE} is rated 20 mating cycles, so break the link at the"
- note added: "channels draws one 0.20 mm track per grounded LV541A pad column straight into that package's thermal pad on F.Cu, before autorouting; Freerouting will not run a track along a row of same-net 0.5"
- note added: "comparator: do not route a raw analog node through it for a timing witness, and do not treat a clean legacy LVC125A capture as LV541A qualification. OE would disable outputs only - it never removes"
- note added: "each need different bias, and pulls that must read HIGH on a switched net reference the switched rail, never the always-on one. Every unused input must be explicitly tied at the board. LV541A at 3.3V"
- note added: "every fault. DEFAULT-ENABLED BY HARDWARE, AND THERE IS NO DISABLE AT ALL: both active-low OE inputs of each package share one net held low by a single 10k pull-down - ${84c143f8-b8f7-412f-b388-3f55d62abdd6:REFERENCE} through ${6c63e654-1b93-4601-99a7-45c9ca25760f:REFERENCE},"
- note added: "findings from this block under the shared rules; a board wanting 0.20 mm inside the block re-routes the block, not the rule (layout conventions 12)."
- note added: "floor(n/2) + floor(n/16), so DIG0 is pin 2 and DIG31 is pin 49, with all 18 grounds on pins 1, 4, 7, 10, 13, 16, 19, 22, 25, 26, 29, 32, 35, 38, 41, 44, 47 and 50. THE MIRROR LIVES ON THE ADAPTER,"
- note added: "input loading or makes a floating input acceptable, which is part of why no mute was fitted. Requires straight-ended 0.30 +/-0.05mm FFC with gold contacts, at least 2mm exposed contact and 3mm"
- note added: "instead tie an unused channel to ground at that via; either way the grounding copper is the board's, never the block's. FLOOR COPPER IS DECLARED: the 0.10 mm gaps between the 32 damping resistors"
- note added: "instrument end."
- note added: "kicad-libs/docs/digital-instrument-port-design-blocks.md under 'No disable control, and why'. DO NOT re-add a control as an oversight fix. Shared 10k is verified against aggregate leakage: 2 x 5uA"
- note added: "leakage against the 0.99 V VIL), so observation works with the MCU in reset or unprogrammed. The contract permits this since 2026-09-15; do not re-add a control as a fix."
- note added: "max gives 0.1V against a 0.99V VIL. If a noise investigation ever needs a mute, detaching the FFC bounds the cable's contribution but NOT the buffers', which keep switching into their board-side traces"
- note added: "maximum even crediting the driver with zero impedance (3.3V/100R = 33mA); 68R gives 49mA, 47R gives 70mA, and the legacy 33R gives 100mA. It is NOT short-circuit protection and does not cover"
- note added: "mm-pitch pads and left those groups unrouted on every camera-board run (layout conventions 11a). Since 2026-09-29 every DIGn also ends at its own escape via above the pad row, so a board may"
- note added: "nameplate value as nominal, not measured. INPUT BIAS IS BOARD-SPECIFIC AND IS NOT IN THIS BLOCK: there is no universal pull-down, because SPI selects, open-drain buses and switched-domain taps"
- note added: "needs VIH >= 2.31V and VIL <= 0.99V with transitions <= 100 ns/V; it is 0-5.5V input tolerant with 2pF typical input capacitance and Ioff <= 5uA at VCC=0. It is NOT Schmitt-triggered and NOT a"
- note added: "no OE port. The owning contract was relaxed on 2026-09-15 from requiring manual disabling to permitting none, so this conforms; the reasoning and the retained future option are in"
- note added: "ns/V, not a Schmitt input. ${32c854d3-e295-4ed0-ae67-c404202c33c2:REFERENCE} to ${97871112-ad18-45a1-a62c-deaacd916849:REFERENCE} (100 nF) bypass each pin 20; ${3b73245c-fad3-495c-87fd-b301079bbe35:REFERENCE} (4.7 uF, X5R 0402, well below nameplate at 3.3 V bias) is the one rail-entry bulk, not a fifth per-package bypass."
- note added: "one per package - so observation works with the MCU held in reset, unprogrammed or unable to boot, and the port cannot be muted without desoldering. There is no manual jumper, no firmware link and"
- note added: "orb_weaver_smd:Texas_RKS0020A_VQFN-20-1EP_2.5x4.5mm_P0.5mm_EP1x3mm, exposed pad 21 to GND), grouped DIG0-7 / DIG8-15 / DIG16-23 / DIG24-31 to match the 13-contact octet windows. The"
- note added: "rail-entry bulk, ${3b73245c-fad3-495c-87fd-b301079bbe35:REFERENCE} / OW-CAP-4U7-0402-X5R-16V, at the supply entry. ${3b73245c-fad3-495c-87fd-b301079bbe35:REFERENCE} is NOT a fifth per-IC bypass - do not 'fix' its distance to any package. Simultaneous-switching budget: 32 x 50pF"
- note added: "reference, enable or stimulus."
- note added: "reference, no enable and no stimulus, and nothing in this block may be driven by the instrument. PIN MAPPING IS THE CONTRACT'S DUT TABLE AND IS NOT MIRRORED: channel n lands on pin 2 + n +"
- note added: "reinforcement; retention-eared cable is NOT qualified for this connector. Rated 20 mating cycles, so prefer breaking the link at the instrument end, and attach or remove the cable with target power off"
- note added: "rotated 180 degrees - delivers DIGn to DIGn. Mirroring both ends cancels and channels arrive as DIG31-n. The ground pattern is palindromic under 51-n, so a mirrored map lands every ground identically"
- note added: "switched rail cannot observe the domain it is powering down with. DECOUPLING is one 100nF per package, ${32c854d3-e295-4ed0-ae67-c404202c33c2:REFERENCE} through ${97871112-ad18-45a1-a62c-deaacd916849:REFERENCE}, hard against each pin 20 with a short return, plus one 4.7uF"
- note added: "unless the actual assembly is hot-plug qualified. Profile is InstrumentPort-Digital-50 draft v0.1, UNQUALIFIED: no measured rate, delay, skew, loading or power-state limit has been established."
- note added: "with the 25/26 double ground at the bank boundary. The mirror lives on instrument_port_digital_50_adapter_ffc_boundary_vertical; mirroring both ends cancels, and ERC and DRC cannot see it."
- note added: "with the connector's ground contacts."
- note added: "within each row."
- note added: "x 3.3V = 5.3nC per all-channel edge, about 1mV of droop against the combined local reservoir. Expect meaningfully less than 4.7uF at 3.3V bias - a 4.7uF X5R in an 0402 derates hard - so treat the"
- note added: "~{OE1}/~{OE2} pull-down,"
- company: Janelia Research Campus -> Orb Weaver
- title: camera-gpio-interface-pcb -> InstrumentPort-Digital-50 DUT boundary, vertical
- moved on the sheet: C501, C502, C503, C504, C505, J501, R501, R502, R503, R504, R505, R506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

Commit message: Regenerate schematics
Parts:
- C502: Placement (none) -> beside ${7e0cdabf-d9e1-4b13-ab00-5a4417fdb564:REFERENCE}.20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
- C503: Placement (none) -> beside ${b1707ec3-0f6f-4e89-a1c4-65233bece57d:REFERENCE}.20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
- C504: Placement (none) -> beside ${69119102-0ebd-473d-a7cb-d952bc88de42:REFERENCE}.20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
- C505: Placement (none) -> beside ${f13cd1d5-28c7-4506-b50d-dbf0bfbd6248:REFERENCE}.20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
- R501: Placement (none) -> beside ${7e0cdabf-d9e1-4b13-ab00-5a4417fdb564:REFERENCE}.1 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
- R502: Placement (none) -> beside ${b1707ec3-0f6f-4e89-a1c4-65233bece57d:REFERENCE}.1 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
- R503: Placement (none) -> beside ${69119102-0ebd-473d-a7cb-d952bc88de42:REFERENCE}.1 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
- R504: Placement (none) -> beside ${f13cd1d5-28c7-4506-b50d-dbf0bfbd6248:REFERENCE}.1 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
Changed lines of the file:
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@@
 			)
 		)
+		(property "Placement" "beside ${7e0cdabf-d9e1-4b13-ab00-5a4417fdb564:REFERENCE}.20 (VCC), on +3.3V"
+			(at 63.5 72.39 0)
+			(hide yes)
+			(show_name no)
+			(do_not_autoplace no)
+			(effects
+				(font
+					(size 1.27 1.27)
+				)
+			)
+		)
 		(pin "1"
 		)
@@
 			)
 		)
+		(property "Placement" "beside ${b1707ec3-0f6f-4e89-a1c4-65233bece57d:REFERENCE}.20 (VCC), on +3.3V"
+			(at 281.94 72.39 0)
+			(hide yes)
+			(show_name no)
+			(do_not_autoplace no)
+			(effects
+				(font
+					(size 1.27 1.27)
+				)
+			)
+		)
 		(pin "1"
 		)
@@
 			)
 		)
+		(property "Placement" "beside ${69119102-0ebd-473d-a7cb-d952bc88de42:REFERENCE}.20 (VCC), on +3.3V"
+			(at 500.38 72.39 0)
+			(hide yes)
+			(show_name no)
+			(do_not_autoplace no)
+			(effects
+				(font
+					(size 1.27 1.27)
+				)
+			)
+		)
 		(pin "1"
 		)
@@
 			)
 		)
+		(property "Placement" "beside ${f13cd1d5-28c7-4506-b50d-dbf0bfbd6248:REFERENCE}.20 (VCC), on +3.3V"
+			(at 63.5 252.73 0)
+			(hide yes)
+			(show_name no)
+			(do_not_autoplace no)
+			(effects
+				(font
+					(size 1.27 1.27)
+				)
+			)
+		)
 		(pin "1"
 		)
@@
 			)
 		)
+		(property "Placement" "beside ${7e0cdabf-d9e1-4b13-ab00-5a4417fdb564:REFERENCE}.1 (~{OE1}), on ~{OE1}"
+			(at 22.86 161.29 0)
+			(hide yes)
+			(show_name no)
+			(do_not_autoplace no)
+			(effects
+				(font
+					(size 1.27 1.27)
+				)
+			)
+		)
 		(pin "1"
 		)
@@
 			)
 		)
+		(property "Placement" "beside ${b1707ec3-0f6f-4e89-a1c4-65233bece57d:REFERENCE}.1 (~{OE1}), on ~{OE2}"
+			(at 241.3 161.29 0)
+			(hide yes)
+			(show_name no)
+			(do_not_autoplace no)
+			(effects
+				(font
+					(size 1.27 1.27)
+				)
+			)
+		)
 		(pin "1"
 		)
@@
 			)
 		)
+		(property "Placement" "beside ${69119102-0ebd-473d-a7cb-d952bc88de42:REFERENCE}.1 (~{OE1}), on ~{OE3}"
+			(at 459.74 161.29 0)
+			(hide yes)
+			(show_name no)
+			(do_not_autoplace no)
+			(effects
+				(font
+					(size 1.27 1.27)
+				)
+			)
+		)
 		(pin "1"
 		)
@@
 			(do_not_autoplace no)
 			(effects
+				(font
+					(size 1.27 1.27)
+				)
+			)
+		)
+		(property "Placement" "beside ${f13cd1d5-28c7-4506-b50d-dbf0bfbd6248:REFERENCE}.1 (~{OE1}), on ~{OE4}"
+			(at 22.86 341.63 0)
+			(hide yes)
+			(show_name no)
+			(do_not_autoplace no)
+			(effects
